File: PCB/ECE477_PCBDesign.kicad_sch (KiCad schematic)
At the start: 0 parts

Commit message: Update Rev 2
Other:
- company: (none) -> ECE477 - Team 4: KayO
- title: (none) -> Hierarchical Sheet
Changed lines of the file:
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@@
 (kicad_sch (version 20230121) (generator eeschema)
   (paper "A3")
+  (title_block
+    (title "Hierarchical Sheet")
+    (date "2024-02-21")
+    (rev "2")
+    (company "ECE477 - Team 4: KayO")
+  )
   (bus (pts (xy 236.22 129.54) (xy 241.3 129.54))
     (stroke (width 0) (type default))
