File: PCB/MCU.kicad_sch (KiCad schematic)
At the start: 2 parts, among them U5 STM32F405RGTx, Y1 24MHz

Commit message: PCB Update - Minh
Parts:
- added C20: 0.47u, symbol Device:C
- added C21, C22, C23, C24, C25, C26: 0.1u, symbol Device:C
- added C27, C28: 20p, symbol Device:C
- added R31: 1k, symbol Device:R
- added R36: R, symbol Device:R
- added R37: 0, symbol Device:R
- added SW5: RST_PB, symbol Switch:SW_Push
- Y1: value 24MHz -> 8MHz
Connections:
- net at Y1.1: now also C28.2, R36.2
- net at Y1.2: now also C27.2, R37.1
- net +3V3: now reaches U5.1 (VBAT)
- net +3V3: now also U5.13 (VDDA), U5.19 (VDD), U5.32 (VDD), U5.48 (VDD), U5.64 (VDD), C21.1, C22.1, C23.1, C24.1, C25.1, C26.1, R31.1
- net GND: now reaches U5.12 (VSSA)
- net GND: now also U5.18 (VSS), U5.63 (VSS), C20.1, C21.2, C22.2, C23.2, C24.2, C25.2, C26.2, C27.1, C28.1, SW5.2
- net STM32.OSC_IN: now reaches U5.5 (PH0)
- net STM32.OSC_IN: now also R37.2
- net STM32.OSC_OUT: now reaches U5.6 (PH1)
- net STM32.OSC_OUT: now also R36.1
- net STM32.NRST: now reaches U5.7 (NRST)
- net STM32.NRST: now also C20.2, R31.2, SW5.1
Other:
- note added: "8MHz HSE OSC_OUT Res depends on Oscillator Characteristic"
- moved on the sheet: Y1

Commit message: update
Parts:
- removed SW5: RST_PB, symbol Switch:SW_Push
- removed U5: STM32F405RGTx, Package_QFP:LQFP-64_10x10mm_P0.5mm, symbol MCU_ST_STM32F4:STM32F405RGTx
- removed Y1: 8MHz, symbol Device:Crystal
- added C310: 2.2u, Capacitor_SMD:C_0603_1608Metric_Pad1.08x0.95mm_HandSolder, symbol Device:C
- added C311, C312: 20p, Capacitor_SMD:C_0603_1608Metric_Pad1.08x0.95mm_HandSolder, symbol Device:C
- added C313, C314, C315: 0.1u, Capacitor_SMD:C_0603_1608Metric_Pad1.08x0.95mm_HandSolder, symbol Device:C
- added D301, D302, D303: D5V0L1B2S9-7, Diode_SMD:D_SOD-923, symbol Device:D_TVS
- added FB301: 120R, Inductor_SMD:L_0603_1608Metric, symbol Device:FerriteBead
- added J301: USB_C_Receptacle_USB2.0_16P, Connector_USB:USB_C_Receptacle_HRO_TYPE-C-31-M-12, symbol Connector:USB_C_Receptacle_USB2.0_16P
- added J302: Conn_01x05_Pin, Connector_PinHeader_2.54mm:PinHeader_1x05_P2.54mm_Vertical, symbol Connector:Conn_01x05_Pin
- added J304: Conn_01x07_Pin, Connector_PinHeader_2.54mm:PinHeader_1x07_P2.54mm_Vertical, symbol Connector:Conn_01x07_Pin
- added R304, R305, R307: 100k, Resistor_SMD:R_0603_1608Metric_Pad0.98x0.95mm_HandSolder, symbol Device:R
- added R306: 10k, Resistor_SMD:R_0603_1608Metric_Pad0.98x0.95mm_HandSolder, symbol Device:R
- added R308, R309, R311: 4.7k, Resistor_SMD:R_0603_1608Metric_Pad0.98x0.95mm_HandSolder, symbol Device:R
- added R310: 2.7k, Resistor_SMD:R_0603_1608Metric_Pad0.98x0.95mm_HandSolder, symbol Device:R
- added R312, R313: 5.1k, Resistor_SMD:R_0603_1608Metric_Pad0.98x0.95mm_HandSolder, symbol Device:R
- added R314, R316: 180, Resistor_SMD:R_0603_1608Metric_Pad0.98x0.95mm_HandSolder, symbol Device:R
- added SW301, SW302: PTS647SM70SMTR2LFS, PTS647SM70SMTR2LFS_CNK, symbol ECE477_PartsLibrary:PTS647SM70SMTR2LFS
- added U301: STM32F411RET6, Package_QFP:LQFP-64_10x10mm_P0.5mm, symbol MCU_ST_STM32F4:STM32F411RETx
- added U302: STM32F103CBT6, Package_QFP:LQFP-48_7x7mm_P0.5mm, symbol MCU_ST_STM32F1:STM32F103CBTx
- added U303: LTST-C155KGJRKT, SON4_LTST-C155KGJRKT_LTO, symbol ECE477_PartsLibrary:LTST-C155KGJRKT
- added X301, X302: CG04874-8M, XTAL_CG04874_NDK, symbol ECE477_PartsLibrary:CG04874-8M
- C301: renamed from C27; footprint (none) -> Capacitor_SMD:C_0603_1608Metric_Pad1.08x0.95mm_HandSolder; DigiKey Part (none) -> 311-1424-1-ND
- C302: renamed from C28; footprint (none) -> Capacitor_SMD:C_0603_1608Metric_Pad1.08x0.95mm_HandSolder; DigiKey Part (none) -> 311-1424-1-ND
- C303: renamed from C20; value 0.47u -> 0.1u; footprint (none) -> Capacitor_SMD:C_0603_1608Metric_Pad1.08x0.95mm_HandSolder; DigiKey Part (none) -> 490-5405-1-ND
- C304: renamed from C21; footprint (none) -> Capacitor_SMD:C_0603_1608Metric_Pad1.08x0.95mm_HandSolder; DigiKey Part (none) -> 490-5405-1-ND
- C305: renamed from C22; footprint (none) -> Capacitor_SMD:C_0603_1608Metric_Pad1.08x0.95mm_HandSolder; DigiKey Part (none) -> 490-5405-1-ND
- C306: renamed from C23; footprint (none) -> Capacitor_SMD:C_0603_1608Metric_Pad1.08x0.95mm_HandSolder; DigiKey Part (none) -> 490-5405-1-ND
- C307: renamed from C24; footprint (none) -> Capacitor_SMD:C_0603_1608Metric_Pad1.08x0.95mm_HandSolder; DigiKey Part (none) -> 490-5405-1-ND
- C308: renamed from C25; footprint (none) -> Capacitor_SMD:C_0603_1608Metric_Pad1.08x0.95mm_HandSolder; DigiKey Part (none) -> 490-5405-1-ND
- C309: renamed from C26; footprint (none) -> Capacitor_SMD:C_0603_1608Metric_Pad1.08x0.95mm_HandSolder; DigiKey Part (none) -> 490-5405-1-ND
- R301: renamed from R31; value 1k -> 100k; footprint (none) -> Resistor_SMD:R_0603_1608Metric_Pad0.98x0.95mm_HandSolder; DigiKey Part (none) -> 311-100KHRCT-ND
- R302: renamed from R37; footprint (none) -> Resistor_SMD:R_0603_1608Metric_Pad0.98x0.95mm_HandSolder; DigiKey Part (none) -> 311-0.0GRCT-ND
- R303: renamed from R36; value R -> 0; footprint (none) -> Resistor_SMD:R_0603_1608Metric_Pad0.98x0.95mm_HandSolder; DigiKey Part (none) -> 311-0.0GRCT-ND
Connections:
- net +3V3: now also J302.1 (Pin_1), J304.1 (Pin_1), R307.1, R308.2, U301.1 (VBAT), U301.13 (VDDA), U301.19 (VDD), U301.32 (VDD), U301.48 (VDD), U301.64 (VDD), U302.1 (VBAT), U302.24 (VDD), U302.36 (VDD), U302.48 (VDD), U302.9 (VDDA), U303.2
- net GND: now also C310.2, C311.1, C312.1, C313.1, C314.2, C315.2, D301.1 (A1), D302.1 (A1), D303.1 (A1), J301.A1 (GND), J301.A12 (GND), J301.B1 (GND), J301.B12 (GND), J301.S1 (SHIELD), J302.3 (Pin_3), J304.3 (Pin_3), R304.1, R305.1, R306.1, R309.1, R311.1, R312.2, R313.1, SW301.3, SW301.4, SW302.3, SW302.4, U301.12 (VSSA), U301.18 (VSS), U301.31 (VSS), U301.47 (VSS), U301.63 (VSS), U302.20 (PB2), U302.23 (VSS), U302.35 (VSS), U302.47 (VSS), U302.8 (VSSA), U303.3
- net at C301.2, R302.1: now also X301.2
- net at C302.2, R303.2: now also X301.1
- net STM32.NRST renamed STM.NRST
- net STM.NRST: now also J302.5 (Pin_5), SW302.1, SW302.2, U301.7 (NRST), U302.18 (PB0)
- net STM32.OSC_IN renamed STM.OSC_IN
- net STM.OSC_IN: now also U301.5 (PH0)
- net STM32.OSC_OUT renamed STM.OSC_OUT
- net STM.OSC_OUT: now also U301.6 (PH1)
- new net: R308.1, R309.2, U302.10 (PA0)
- new net: R305.2, U302.44 (BOOT0)
- new net: J301.A5 (CC1), R312.1
- new net: R310.1, R311.2, U302.39 (PB3)
- new net: J301.B5 (CC2), R313.2
- new net: R306.2, U302.2 (PC13)
- new net: R314.2, U303.1
- new net: R316.2, U303.4
- new net: C310.1, U301.30 (VCAP1)
- new net: R304.2, U301.60 (BOOT0)
- new net +5V: C315.1, D303.2 (A2), FB301.2, R310.2
- new net BAT.EN1: U301.37 (PC6)
- new net BAT.EN2: U301.38 (PC7)
- new net BAT.GPOUT: U301.39 (PC8)
- new net BAT.TMR: U301.42 (PA9)
- new net BAT.~{CE}: U301.43 (PA10)
- new net BT.GPIO3: U301.20 (PA4)
- new net BT.GPIO4: U301.21 (PA5)
- new net BT.GPIO6: U301.22 (PA6)
- new net BT.GPIO7: U301.23 (PA7)
- new net BT.RX: U301.17 (PA3)
- new net BT.TX: U301.16 (PA2)
- new net I2C.SCL: U301.41 (PA8)
- new net I2C.SDA: U301.40 (PC9)
- new net KEY.B17: U301.61 (PB8)
- new net KEY.B18: U301.62 (PB9)
- new net KEY.COL0: U301.26 (PB0)
- new net KEY.COL1: U301.27 (PB1)
- new net KEY.COL2: U301.28 (PB2)
- new net KEY.COL3: U301.55 (PB3)
- new net KEY.ROW0: U301.56 (PB4)
- new net KEY.ROW1: U301.57 (PB5)
- new net KEY.ROW2: U301.58 (PB6)
- new net KEY.ROW3: U301.59 (PB7)
- new net LCD.DC: U301.52 (PC11)
- new net LCD.MOSI: U301.53 (PC12)
- new net LCD.SCLK: U301.51 (PC10)
- new net LCD.~{CS}: U301.50 (PA15)
- new net LCD.~{RST}: U301.54 (PD2)
- new net SD.CD: U301.29 (PB10)
- new net SD.MISO: U301.35 (PB14)
- new net SD.MOSI: U301.36 (PB15)
- new net SD.SCLK: U301.34 (PB13)
- new net SD.~{CS}: U301.33 (PB12)
- new net STLink.D+: D301.2 (A2), J301.A6 (D+), J301.B6 (D+), U302.33 (PA12)
- new net STLink.D-: D302.2 (A2), J301.A7 (D-), J301.B7 (D-), U302.32 (PA11)
- new net STLink.LED: R314.1, R316.1, U302.30 (PA9)
- new net STLink.NRST: C313.2, J304.5 (Pin_5), R307.2, SW301.1, SW301.2, U302.7 (NRST)
- new net STLink.OSC_IN: C311.2, U302.5 (PD0), X302.2
- new net STLink.OSC_OUT: C312.2, U302.6 (PD1), X302.1
- new net STLink.RX: J304.7 (Pin_7), U302.12 (PA2)
- new net STLink.SWCLK: J304.2 (Pin_2), U302.37 (PA14)
- new net STLink.SWDIO: J304.4 (Pin_4), U302.34 (PA13)
- new net STLink.TX: J304.6 (Pin_6), U302.13 (PA3)
- new net STM.SWCLK: J302.2 (Pin_2), U301.49 (PA14), U302.26 (PB13)
- new net STM.SWDIO: J302.4 (Pin_4), U301.46 (PA13), U302.27 (PB14)
- new net USB.D+: U301.45 (PA12)
- new net USB.D-: U301.44 (PA11)
- new net USB.Detect: U301.25 (PC5)
- new net V_RAW_STLink: C314.1, FB301.1, J301.A4 (VBUS), J301.A9 (VBUS), J301.B4 (VBUS), J301.B9 (VBUS)
- no-connect marks 0 -> 33
Other:
- note added: "STLink"
- note added: "STM32 MCU"
- note added: "USB PWR Filtering"
- note added: "USB_C"
- moved on the sheet: C301, C302, C303, C304, C305, C306, C307, C308, C309, R301, R302, R303

Commit message: Update 90% done
Parts:
- removed D301, D302: D5V0L1B2S9-7, Diode_SMD:D_SOD-923, symbol Device:D_TVS
- removed J301: USB_C_Receptacle_USB2.0_16P, Connector_USB:USB_C_Receptacle_HRO_TYPE-C-31-M-12, symbol Connector:USB_C_Receptacle_USB2.0_16P
- removed J302: Conn_01x05_Pin, Connector_PinHeader_2.54mm:PinHeader_1x05_P2.54mm_Vertical, symbol Connector:Conn_01x05_Pin
- removed J304: Conn_01x07_Pin, Connector_PinHeader_2.54mm:PinHeader_1x07_P2.54mm_Vertical, symbol Connector:Conn_01x07_Pin
- removed R312, R313: 5.1k, Resistor_SMD:R_0603_1608Metric_Pad0.98x0.95mm_HandSolder, symbol Device:R
- added C316, C317, C318, C319, C320: 0.1u, Capacitor_SMD:C_0603_1608Metric_Pad1.08x0.95mm_HandSolder, symbol Device:C
- added D302: 3757-SS12L_R1_00001CT-ND, Diode_SMD:D_SMA, symbol Device:D_Schottky
- added J302: Conn_01x03_Pin, Connector_PinHeader_2.54mm:PinHeader_1x03_P2.54mm_Vertical, symbol Connector:Conn_01x03_Pin
- added J303: STLink Connector, ECE477_PartsLibrary:CONN10_302-S101_OST, symbol Connector_Generic:Conn_02x05_Odd_Even
- added SW303: SW_DPDT_x2, ECE477_PartsLibrary:SW_JS202011SCQN, symbol Switch:SW_DPDT_x2
- added SW305: 1-1825010-3, ECE477_PartsLibrary:SW_1-1825010-3, symbol ECE477_PartsLibrary:1-1825010-3
- C301: renamed from C304; Manufacturer (none) -> Murata Electronics; Mfg. Part # (none) -> GRM033R61A104ME15D; Package (none) -> 0603; Supplier (none) -> DigiKey; Supplier Part # (none) -> 490-5405-1-ND
- C302: renamed from C305; Manufacturer (none) -> Murata Electronics; Mfg. Part # (none) -> GRM033R61A104ME15D; Package (none) -> 0603; Supplier (none) -> DigiKey; Supplier Part # (none) -> 490-5405-1-ND
- C303: renamed from C301; Manufacturer (none) -> YAGEO; Mfg. Part # (none) -> CC0603JRNPO9BN200; Package (none) -> 0603; Supplier (none) -> DigiKey; Supplier Part # (none) -> 311-1424-1-ND
- C304: renamed from C302; Manufacturer (none) -> YAGEO; Mfg. Part # (none) -> CC0603JRNPO9BN200; Package (none) -> 0603; Supplier (none) -> DigiKey; Supplier Part # (none) -> 311-1424-1-ND
- C305: renamed from C306; Manufacturer (none) -> Murata Electronics; Mfg. Part # (none) -> GRM033R61A104ME15D; Package (none) -> 0603; Supplier (none) -> DigiKey; Supplier Part # (none) -> 490-5405-1-ND
- C306: renamed from C303; Manufacturer (none) -> Murata Electronics; Mfg. Part # (none) -> GRM033R61A104ME15D; Package (none) -> 0603; Supplier (none) -> DigiKey; Supplier Part # (none) -> 490-5405-1-ND
- C307, C308, C309, C313, C314, C315: Manufacturer (none) -> Murata Electronics; Mfg. Part # (none) -> GRM033R61A104ME15D; Package (none) -> 0603; Supplier (none) -> DigiKey; Supplier Part # (none) -> 490-5405-1-ND
- C310: Manufacturer (none) -> Murata Electronics; Mfg. Part # (none) -> GRM188R61E225KA12D; Package (none) -> 0603; Supplier (none) -> DigiKey; Supplier Part # (none) -> 490-10731-1-ND
- C311, C312: Manufacturer (none) -> YAGEO; Mfg. Part # (none) -> CC0603JRNPO9BN200; Package (none) -> 0603; Supplier (none) -> DigiKey; Supplier Part # (none) -> 311-1424-1-ND
- D301: renamed from D303; value D5V0L1B2S9-7 -> D5V0L1B2T-7; footprint Diode_SMD:D_SOD-923 -> Diode_SMD:D_SOD-523; DigiKey Part D5V0L1B2S9-7DICT-ND -> D5V0L1B2T-7DICT-ND; Manufacturer (none) -> Diodes Incorporated; Mfg. Part # (none) -> D5V0L1B2T-7; Package (none) -> SOD-523; Supplier (none) -> DigiKey; Supplier Part # (none) -> D5V0L1B2T-7DICT-ND
- FB301: Manufacturer (none) -> Murata Electronics; Mfg. Part # (none) -> BLM18BD121SH1D; Package (none) -> 0603; Supplier (none) -> DigiKey; Supplier Part # (none) -> 490-17710-1-ND
- R301, R304: Manufacturer (none) -> YAGEO; Mfg. Part # (none) -> RC0603FR-07100KL; Package (none) -> 0603; Supplier (none) -> DigiKey; Supplier Part # (none) -> 311-100KHRCT-ND
- R302, R303: Manufacturer (none) -> YAGEO; Mfg. Part # (none) -> RC0603JR-070RL; Package (none) -> 0603; Supplier (none) -> DigiKey; Supplier Part # (none) -> 311-0.0GRCT-ND
- R305: renamed from R307; Manufacturer (none) -> YAGEO; Mfg. Part # (none) -> RC0603FR-07100KL; Package (none) -> 0603; Supplier (none) -> DigiKey; Supplier Part # (none) -> 311-100KHRCT-ND
- R306: renamed from R311; Manufacturer (none) -> YAGEO; Mfg. Part # (none) -> RC0603FR-074K7L; Package (none) -> 0603; Supplier (none) -> DigiKey; Supplier Part # (none) -> 311-4.70KHRCT-ND
- R307: renamed from R310; Manufacturer (none) -> RMCF0603FT2K70; Mfg. Part # (none) -> RMCF0603FT2K70; Package (none) -> 0603; Supplier (none) -> DigiKey; Supplier Part # (none) -> RMCF0603FT2K70CT-ND
- R308: renamed from R306; Manufacturer (none) -> YAGEO; Mfg. Part # (none) -> RC0603JR-0710KL; Package (none) -> 0603; Supplier (none) -> DigiKey; Supplier Part # (none) -> 311-10KGRCT-ND
- R309: renamed from R305; Manufacturer (none) -> YAGEO; Mfg. Part # (none) -> RC0603FR-07100KL; Package (none) -> 0603; Supplier (none) -> DigiKey; Supplier Part # (none) -> 311-100KHRCT-ND
- R310: renamed from R314; Manufacturer (none) -> YAGEO; Mfg. Part # (none) -> RC0603FR-13180RL; Package (none) -> 0603; Supplier (none) -> DigiKey; Supplier Part # (none) -> 13-RC0603FR-13180RLCT-ND
- R311: renamed from R316; Manufacturer (none) -> YAGEO; Mfg. Part # (none) -> RC0603FR-13180RL; Package (none) -> 0603; Supplier (none) -> DigiKey; Supplier Part # (none) -> 13-RC0603FR-13180RLCT-ND
- R312: renamed from R308; Manufacturer (none) -> YAGEO; Mfg. Part # (none) -> RC0603FR-074K7L; Package (none) -> 0603; Supplier (none) -> DigiKey; Supplier Part # (none) -> 311-4.70KHRCT-ND
- R313: renamed from R309; Manufacturer (none) -> YAGEO; Mfg. Part # (none) -> RC0603FR-074K7L; Package (none) -> 0603; Supplier (none) -> DigiKey; Supplier Part # (none) -> 311-4.70KHRCT-ND
- SW301: renamed from SW302; footprint PTS647SM70SMTR2LFS_CNK -> ECE477_PartsLibrary:PTS647SM70SMTR2LFS_CNK; Manufacturer (none) -> C&K; Mfg. Part # (none) -> PTS 647 SM70 SMTR2 LFS; Package (none) -> PTS647SM70SMTR2LFS_CNK; Supplier (none) -> DigiKey; Supplier Part # (none) -> PTS647SM70SMTR2LFSCT-ND
- SW302: renamed from SW301; footprint PTS647SM70SMTR2LFS_CNK -> ECE477_PartsLibrary:PTS647SM70SMTR2LFS_CNK; Manufacturer (none) -> C&K; Mfg. Part # (none) -> PTS 647 SM70 SMTR2 LFS; Package (none) -> PTS647SM70SMTR2LFS_CNK; Supplier (none) -> DigiKey; Supplier Part # (none) -> PTS647SM70SMTR2LFSCT-ND
- U301: Manufacturer (none) -> STMicroelectronics; Mfg. Part # (none) -> STM32F411RET6; Package (none) -> 64-LQFP; Supplier (none) -> DigiKey; Supplier Part # (none) -> 497-14909-ND
- U302: Manufacturer (none) -> STMicroelectronics; Mfg. Part # (none) -> STM32F103CBT6; Package (none) -> 48-LQFP; Supplier (none) -> DigiKey; Supplier Part # (none) -> 497-6288-ND
- U303: footprint SON4_LTST-C155KGJRKT_LTO -> ECE477_PartsLibrary:SON4_LTST-C155KGJRKT_LTO; Manufacturer (none) -> LITEON; Mfg. Part # (none) -> LTST-C155KGJRKT; Package (none) -> 1210; Supplier (none) -> DigiKey; Supplier Part # (none) -> 160-1409-1-ND
- X301, X302: footprint XTAL_CG04874_NDK -> ECE477_PartsLibrary:XTAL_CG04874_NDK; Manufacturer (none) -> NDK America, Inc.; Mfg. Part # (none) -> CG04874-8M; Package (none) -> 2-SMD, No Lead; Supplier (none) -> DigiKey; Supplier Part # (none) -> 644-CG04874-8MCT-ND
Connections:
- net +3V3: now also C316.1, C317.1, C318.1, C319.1, C320.1
- net GND: now also C316.2, C317.2, C318.2, C319.2, C320.2, J302.3 (Pin_3), J303.3 (Pin_3), J303.4 (Pin_4)
- net STLink.D+: now also SW303.4 (C)
- net STLink.D-: now also SW303.3 (C)
- net STLink.NRST: now also SW305.3
- net STLink.RX: now also J302.2 (Pin_2)
- net STLink.SWCLK: now also SW305.6
- net STLink.SWDIO: now also SW305.10
- net STLink.TX: now also J302.1 (Pin_1)
- net STM.NRST: now also SW305.1
- net STM.SWCLK: now also SW305.4
- net STM.SWDIO: now also SW305.12
- net USB.D+: now also SW303.5 (B); no longer U301.45 (PA12)
- net USB.D-: now also SW303.2 (B); no longer U301.44 (PA11)
- net V_RAW_STLink: now also D302.2 (A), J303.10 (Pin_10), J303.9 (Pin_9); no longer FB301.1
- new net: D302.1 (K), FB301.1
- new net JT.NRST: J303.1 (Pin_1), SW305.2
- new net JT.SWCLK: J303.6 (Pin_6), SW305.5
- new net JT.SWDIO: J303.2 (Pin_2), SW305.11
- new net STM.D+: SW303.6 (A), U301.45 (PA12)
- new net STM.D-: SW303.1 (A), U301.44 (PA11)
- no-connect marks 33 -> 37
Other:
- note added: "USB Mode Switch - Turn on to program the main STM32"
- note removed: "USB_C"
- moved on the sheet: C315, D301, FB301

Commit message: design 02/17
Parts:
- added D303, D304: Debug_LED, Diode_SMD:D_0805_2012Metric_Pad1.15x1.40mm_HandSolder, symbol Device:LED
- added Q301: S9013, Package_TO_SOT_SMD:SOT-23-3, symbol Transistor_BJT:2N2219
- added R314, R315: 250, Resistor_SMD:R_0603_1608Metric_Pad0.98x0.95mm_HandSolder, symbol Device:R
- added R316, R318: 100, Resistor_SMD:R_0603_1608Metric_Pad0.98x0.95mm_HandSolder, symbol Device:R
- added R317, R319: 10k, Resistor_SMD:R_0603_1608Metric_Pad0.98x0.95mm_HandSolder, symbol Device:R
- added R320: 39k, Resistor_SMD:R_0603_1608Metric_Pad0.98x0.95mm_HandSolder, symbol Device:R
- added R321: 1k5, Resistor_SMD:R_0603_1608Metric_Pad0.98x0.95mm_HandSolder, symbol Device:R
Connections:
- net +3V3: now also Q301.3 (C)
- net +5V: now also R319.1
- net GND: now also R314.1, R315.1, R317.2, R320.2
- net STLink.D+: now also R321.2
- net STM.SWCLK: now also U302.15 (PA5)
- net STM.SWDIO: now also R316.1
- net at U301.14 (PA0): now also D303.2 (A)
- net at U301.15 (PA1): now also D304.2 (A)
- net at U302.25 (PB12): now also R316.2
- net at U302.3 (PC14): now also R317.1
- net STLink.RENUM: now reaches U302.38 (PA15)
- net STLink.RENUM: now also R318.2
- new net: Q301.1 (E), R321.1
- new net: Q301.2 (B), R318.1, R319.2, R320.1
- new net: D304.1 (K), R315.2
- new net: D303.1 (K), R314.2
- no-connect marks 37 -> 31
Other:
- moved on the sheet: C314, C315, D301, D302, FB301, R306, R307

Commit message: Update Rev 2
Parts:
- removed C311, C312: 20p, Capacitor_SMD:C_0603_1608Metric_Pad1.08x0.95mm_HandSolder, symbol Device:C
- removed J302: Conn_01x03_Pin, Connector_PinHeader_2.54mm:PinHeader_1x03_P2.54mm_Vertical, symbol Connector:Conn_01x03_Pin
- removed R302, R303: 0, Resistor_SMD:R_0603_1608Metric_Pad0.98x0.95mm_HandSolder, symbol Device:R
- removed SW305: 1-1825010-3, ECE477_PartsLibrary:SW_1-1825010-3, symbol ECE477_PartsLibrary:1-1825010-3
- removed X301, X302: CG04874-8M, ECE477_PartsLibrary:XTAL_CG04874_NDK, symbol ECE477_PartsLibrary:CG04874-8M
- added J301: Conn_01x03_Pin, Connector_PinHeader_2.54mm:PinHeader_1x03_P2.54mm_Vertical, symbol Connector:Conn_01x03_Pin
- added J302: Conn_01x10_Pin, Connector_PinHeader_2.54mm:PinHeader_1x07_P2.54mm_Vertical, symbol Connector:Conn_01x07_Pin
- added U304, U305: MAX7375AXR805, Package_TO_SOT_SMD:SOT-323_SC-70, symbol Oscillator:MAX7375AXR805
- C303, C304: value 20p -> 0.1u; DigiKey Part 311-1424-1-ND -> 490-5405-1-ND; Manufacturer YAGEO -> Murata Electronics; Mfg. Part # CC0603JRNPO9BN200 -> GRM033R61A104ME15D; Supplier Part # 311-1424-1-ND -> 490-5405-1-ND
Connections:
- net BAT.EN2 is gone; now on net BAT.~{CE}: U301.38 (PC7)
- net JT.NRST is gone; now on net STM.NRST: J303.1 (Pin_1)
- net JT.SWCLK is gone; now on net STM.SWCLK: J303.6 (Pin_6)
- net JT.SWDIO is gone; now on net STM.SWDIO: J303.2 (Pin_2)
- net +3V3: now also C303.2, C304.2, U304.1 (V+), U305.1 (V+)
- net BAT.~{CE}: no longer U301.43 (PA10)
- net GND: now also J301.3 (Pin_3), J302.3 (Pin_3), U304.3 (GND), U305.3 (GND)
- net STLink.NRST: now also J302.1 (Pin_1)
- net STLink.OSC_IN: now also U305.2 (CLOCK)
- net STLink.RX: now also J302.7 (Pin_7)
- net STLink.SWCLK: now also J302.4 (Pin_4)
- net STLink.SWDIO: now also J302.2 (Pin_2)
- net STLink.TX: now also J302.6 (Pin_6)
- net STM.OSC_IN: now also U304.2 (CLOCK)
- net V_RAW_STLink: now also J302.5 (Pin_5)
- net BAT.EN1: no longer names the net of U301.37 (PC6)
- net BAT.TMR renamed Debug.TX
- net Debug.TX: now also J301.2 (Pin_2)
- net BT.GPIO3: no longer names the net of U301.20 (PA4)
- net BT.GPIO4: no longer names the net of U301.21 (PA5)
- net BT.GPIO6: no longer names the net of U301.22 (PA6)
- net BT.GPIO7: no longer names the net of U301.23 (PA7)
- net STLink.OSC_OUT: no longer names the net of U302.6 (PD1)
- net STM.OSC_OUT: no longer names the net of U301.6 (PH1)
- new net Debug.RX: J301.1 (Pin_1), U301.43 (PA10)
- no-connect marks 31 -> 35
Other:
- note added: "STM32F411 IO Map"
- company: (none) -> ECE477 - Team 4: KayO
- title: (none) -> MCU
- moved on the sheet: C313, J303, R305, R310, R311, SW302, U303
