File: PCB/MCU.kicad_sch (KiCad schematic)
At the start: 56 parts, among them J301 Conn_01x03_Pin, J302 Conn_01x10_Pin, J303 STLink Connector, J304 Conn_01x03_Pin, J305 Conn_01x03_Pin, Q301 S9013, SW301 PTS647SM70SMTR2LFS, SW302 PTS647SM70SMTR2LFS, SW303 SW_DPDT_x2, U301 STM32F411RET6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

Commit message: PCB Update
Parts:
- added J306: Conn_01x03_Pin, Connector_PinHeader_2.54mm:PinHeader_1x03_P2.54mm_Vertical, symbol Connector:Conn_01x03_Pin
- D301: value D5V0L1B2T-7 -> D5V0L1B2WS-7; footprint Diode_SMD:D_SOD-523 -> Diode_SMD:D_SOD-323_HandSoldering; Mfg. Part # D5V0L1B2T-7 -> D5V0L1B2WS-7; Supplier Part # D5V0L1B2T-7DICT-ND -> D5V0L1B2WS-7DICT-ND
Connections:
- net at U301.2 (PC13): now also J306.1 (Pin_1)
- net at U301.3 (PC14): now also J306.2 (Pin_2)
- net at U301.4 (PC15): now also J306.3 (Pin_3)
- no-connect marks 34 -> 31
Changed lines of the file:
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@@
   (junction (at 262.89 262.89) (diameter 0) (color 0 0 0 0)
   )
-  (no_connect (at 115.57 97.79))
-  (no_connect (at 115.57 100.33))
   (no_connect (at 279.4 92.71))
   (no_connect (at 81.28 135.255))
@@
   (no_connect (at 115.57 77.47))
   (no_connect (at 312.42 44.45))
-  (no_connect (at 115.57 95.25))
   (no_connect (at 115.57 69.85))
   (no_connect (at 151.13 57.15))
@@
     (stroke (width 0) (type default))
   )
+  (wire (pts (xy 94.615 100.33) (xy 115.57 100.33))
+    (stroke (width 0) (type default))
+  )
   (wire (pts (xy 229.87 158.115) (xy 229.87 154.305))
     (stroke (width 0) (type default))
@@
     (stroke (width 0) (type default))
   )
+  (wire (pts (xy 94.615 97.79) (xy 115.57 97.79))
+    (stroke (width 0) (type default))
+  )
   (wire (pts (xy 297.18 34.29) (xy 297.18 35.56))
     (stroke (width 0) (type default))
@@
     (stroke (width 0) (type default))
   )
+  (wire (pts (xy 94.615 95.25) (xy 115.57 95.25))
+    (stroke (width 0) (type default))
+  )
   (wire (pts (xy 114.3 57.15) (xy 115.57 57.15))
     (stroke (width 0) (type default))
@@
     )
   )
+  (symbol (lib_id "Connector:Conn_01x03_Pin") (at 89.535 97.79 0) (unit 1)
+    (in_bom no) (on_board yes) (dnp no) (fields_autoplaced)
+    (property "Reference" "J306" (at 90.17 90.17 0)
+      (effects (font (size 1.27 1.27)))
+    )
+    (property "Value" "Conn_01x03_Pin" (at 90.17 92.71 0)
+      (effects (font (size 1.27 1.27)))
+    )
+    (property "Footprint" "Connector_PinHeader_2.54mm:PinHeader_1x03_P2.54mm_Vertical" (at 89.535 97.79 0)
+      (effects (font (size 1.27 1.27)) hide)
+    )
+    (property "Datasheet" "~" (at 89.535 97.79 0)
+      (effects (font (size 1.27 1.27)) hide)
+    )
+    (property "Description" "" (at 89.535 97.79 0)
+      (effects (font (size 1.27 1.27)) hide)
+    )
+    (property "Manufacturer" "" (at 89.535 97.79 0)
+      (effects (font (size 1.27 1.27)) hide)
+    )
+    (property "Mfg. Part #" "" (at 89.535 97.79 0)
+      (effects (font (size 1.27 1.27)) hide)
+    )
+    (property "Supplier" "N/A" (at 89.535 97.79 0)
+      (effects (font (size 1.27 1.27)) hide)
+    )
+    (property "Supplier Part #" "" (at 89.535 97.79 0)
+      (effects (font (size 1.27 1.27)) hide)
+    )
+    (pin "2")
+    (pin "3")
+    (pin "1")
+    (instances
+      (project "ECE477_PCBDesign"
+        (path "/a3f06f97-9851-42dd-ac9b-8261120cb59a/e3668cda-1f90-422e-8fca-715d2e2d8332"
+          (reference "J306") (unit 1)
+        )
+      )
+    )
+  )
   (symbol (lib_id "power:GND") (at 326.39 41.91 0) (unit 1)
     (in_bom yes) (on_board yes) (dnp no)
@@
       (effects (font (size 1.27 1.27)) (justify left))
     )
-    (property "Value" "D5V0L1B2T-7" (at 276.86 267.97 90)
+    (property "Value" "D5V0L1B2WS-7" (at 276.86 267.97 90)
       (effects (font (size 1.27 1.27)) (justify left))
     )
-    (property "Footprint" "Diode_SMD:D_SOD-523" (at 274.32 259.08 0)
+    (property "Footprint" "Diode_SMD:D_SOD-323_HandSoldering" (at 274.32 259.08 0)
       (effects (font (size 1.27 1.27)) hide)
     )
@@
       (effects (font (size 1.27 1.27)) hide)
     )
-    (property "Mfg. Part #" "D5V0L1B2T-7" (at 274.32 259.08 0)
+    (property "Mfg. Part #" "D5V0L1B2WS-7" (at 274.32 259.08 0)
       (effects (font (size 1.27 1.27)) hide)
     )
@@
       (effects (font (size 1.27 1.27)) hide)
     )
-    (property "Supplier Part #" "D5V0L1B2T-7DICT-ND" (at 274.32 259.08 0)
+    (property "Supplier Part #" "D5V0L1B2WS-7DICT-ND" (at 274.32 259.08 0)
       (effects (font (size 1.27 1.27)) hide)
     )
