File: PCB/PSU.kicad_sch (KiCad schematic)
At the start: 72 parts, among them J2 Conn_01x02_Pin, J3 USB_C_Receptacle_USB2.0, J4 Conn_01x02_Pin, Q1 BC817, Q2 BC817, Q3 BC817, Q4 BC817, Q6 2N2219, SW2 SW_SPDT, SW3 SW_DPDT_x2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

Commit message: PCB init - Minh
Parts:
- added D13: 3VDetect_LED, Diode_SMD:D_0402_1005Metric_Pad0.77x0.64mm_HandSolder, symbol Device:LED
- added R25: 470, symbol Device:R
- added R26: 250, symbol Device:R
- added U7: LMS33460MG, LMS33460MG:SOT65P210X110-5N, symbol ECE477_PartsLibrary:LMS33460MG
Connections:
- net GND: now also D13.1 (K), U7.2 (GND), U7.3 (GND__1)
- net SYS.PWR: now also R25.1, U7.5 (VIN)
- new net: R25.2, R26.1, U7.4 (~{VOUT})
- new net: D13.2 (A), R26.2
Other:
- note added: "Below 3V Detection (>3V -> LED off)"
- note removed: "Low Power Detect"
- moved on the sheet: D12, R7, SW3B

Commit message: PCB update - Minh
Connections:
- net BAT.SCL renamed I2C.SCL
- net BAT.SDA renamed I2C.SDA
Changed lines of the file:
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@@
     (stroke (width 0) (type default))
   )
-  (bus (pts (xy 375.92 234.95) (xy 373.38 234.95))
+  (bus (pts (xy 367.03 232.41) (xy 364.49 232.41))
     (stroke (width 0) (type default))
   )
@@
     (stroke (width 0) (type default))
   )
+  (bus (pts (xy 347.98 240.03) (xy 356.87 240.03))
+    (stroke (width 0) (type default))
+  )
   (wire (pts (xy 50.8 69.85) (xy 53.975 69.85))
     (stroke (width 0) (type default))
@@
     (stroke (width 0) (type default))
   )
-  (bus (pts (xy 375.92 238.76) (xy 375.92 234.95))
+  (bus (pts (xy 367.03 236.22) (xy 367.03 232.41))
     (stroke (width 0) (type default))
   )
@@
     (stroke (width 0) (type default))
   )
-  (bus (pts (xy 375.92 238.76) (xy 372.11 238.76))
+  (bus (pts (xy 367.03 236.22) (xy 363.22 236.22))
     (stroke (width 0) (type default))
   )
@@
     )
   )
-  (global_label "BAT.SDA" (shape input) (at 168.91 53.34 0) (fields_autoplaced)
+  (global_label "I2C.SDA" (shape input) (at 168.91 53.34 0) (fields_autoplaced)
     (effects (font (size 1.27 1.27)) (justify left))
-    (property "Intersheetrefs" "${INTERSHEET_REFS}" (at 179.3943 53.34 0)
+    (property "Intersheetrefs" "${INTERSHEET_REFS}" (at 179.1524 53.34 0)
       (effects (font (size 1.27 1.27)) (justify left) hide)
     )
   )
-  (global_label "BAT.SCL" (shape input) (at 168.91 50.8 0) (fields_autoplaced)
+  (global_label "I2C.SCL" (shape input) (at 168.91 50.8 0) (fields_autoplaced)
     (effects (font (size 1.27 1.27)) (justify left))
-    (property "Intersheetrefs" "${INTERSHEET_REFS}" (at 179.3338 50.8 0)
+    (property "Intersheetrefs" "${INTERSHEET_REFS}" (at 179.0919 50.8 0)
       (effects (font (size 1.27 1.27)) (justify left) hide)
     )
@@
     )
   )
-  (global_label "BAT{SCL, SDA, OFF, ~{CE}, TMR, EN1, EN2, GPOUT}" (shape input) (at 373.38 234.95 180) (fields_autoplaced)
+  (global_label "BAT{OFF, ~{CE}, TMR, EN1, EN2, GPOUT}" (shape input) (at 364.49 232.41 180) (fields_autoplaced)
     (effects (font (size 1.27 1.27)) (justify right))
-    (property "Intersheetrefs" "${INTERSHEET_REFS}" (at 324.1304 234.95 0)
+    (property "Intersheetrefs" "${INTERSHEET_REFS}" (at 325.4609 232.41 0)
       (effects (font (size 1.27 1.27)) (justify right) hide)
     )
@@
     )
   )
+  (global_label "I2C{SCL, SDA}" (shape input) (at 347.98 240.03 180) (fields_autoplaced)
+    (effects (font (size 1.27 1.27)) (justify right))
+    (property "Intersheetrefs" "${INTERSHEET_REFS}" (at 331.569 240.03 0)
+      (effects (font (size 1.27 1.27)) (justify right) hide)
+    )
+  )
   (global_label "BAT.EN2" (shape input) (at 304.8 115.57 180) (fields_autoplaced)
     (effects (font (size 1.27 1.27)) (justify right))
@@
     (effects (font (size 1.27 1.27)) (justify left))
   )
-  (hierarchical_label "BAT{SCL, SDA, OFF, ~{CE}, TMR, EN1, EN2, GPOUT}" (shape input) (at 372.11 238.76 180) (fields_autoplaced)
+  (hierarchical_label "BAT{OFF, ~{CE}, TMR, EN1, EN2, GPOUT}" (shape input) (at 363.22 236.22 180) (fields_autoplaced)
     (effects (font (size 1.27 1.27)) (justify right))
   )
+  (hierarchical_label "I2C{SCL, SDA}" (shape input) (at 356.87 240.03 0) (fields_autoplaced)
+    (effects (font (size 1.27 1.27)) (justify left))
+  )
   (symbol (lib_id "Device:C") (at 111.76 115.57 0) (mirror y) (unit 1)
