File: PCB/PSU.kicad_sch (KiCad schematic)
At the start: 76 parts, among them J2 Conn_01x02_Pin, J3 USB_C_Receptacle_USB2.0, J4 Conn_01x02_Pin, Q1 BC817, Q2 BC817, Q3 BC817, Q4 BC817, Q6 2N2219, SW2 SW_SPDT, SW3 SW_DPDT_x2, U1 BQ24075RGT, U2 BQ27441DRZR-G1A, U3 TPS63031DSK, U6 TPS63021DSJR, U7 LMS33460MG

Commit message: update
Parts:
- removed C10: 0.1u, symbol Device:C
- removed C11, C12, C13: 22u, symbol Device:C
- removed C9: 10u, symbol Device:C
- removed D11, D6, D7, D8, D9: BZX84Cxx, Package_TO_SOT_SMD:SOT-23, symbol Diode:BZX84Cxx
- removed J3: USB_C_Receptacle_USB2.0, Connector_USB:USB_C_Receptacle_HRO_TYPE-C-31-M-12, symbol Connector:USB_C_Receptacle_USB2.0
- removed JP1, JP2: Jumper_2_Bridged, symbol Jumper:Jumper_2_Bridged
- removed JP3, JP5: Jumper_2_Open, symbol Jumper:Jumper_2_Open
- removed L1, L2: 1.5u, symbol Device:L
- removed Q2, Q3, Q4: BC817, Package_TO_SOT_SMD:SOT-23, symbol Transistor_BJT:BC817
- removed Q6: 2N2219, Package_TO_SOT_THT:TO-39-3, symbol Transistor_BJT:2N2219
- removed R21: 100k, symbol Device:R
- removed R22, R24: 1M, symbol Device:R
- removed R23: 180k, symbol Device:R
- removed SW2: SW_SPDT, symbol Switch:SW_SPDT
- removed SW3: SW_DPDT_x2, symbol Switch:SW_DPDT_x2
- removed U6: TPS63021DSJR, TPS63021DSJR:IC_TPS63021DSJR, symbol ECE477_PartsLibrary:TPS63021DSJR
- added C208: 22u, Capacitor_SMD:C_0603_1608Metric_Pad1.08x0.95mm_HandSolder, symbol Device:C
- added C211, C212: 0.1u, Capacitor_SMD:C_0603_1608Metric_Pad1.08x0.95mm_HandSolder, symbol Device:C
- added D206: D5V0L1B2S9-7, Diode_SMD:D_SOD-923, symbol Device:D_TVS
- added FB201: 120R, Inductor_SMD:L_0603_1608Metric, symbol Device:FerriteBead
- added J204: USB_C_Receptacle_USB2.0_16P, Connector_USB:USB_C_Receptacle_HRO_TYPE-C-31-M-12, symbol Connector:USB_C_Receptacle_USB2.0_16P
- added JP201, JP203: Jumper_2_Open, symbol Jumper:Jumper_2_Open
- added JP202, JP204: Jumper_2_Bridged, symbol Jumper:Jumper_2_Bridged
- added L202: 1.5u, IND_TAIYO_NR3015_TAY, symbol ECE477_PartsLibrary:NR3015T1R5N
- added L203: 0.47u, IND_IHLP-2020CZ, symbol ECE477_PartsLibrary:IHLP2020CZERR47M11
- added Q201, Q203, Q204, Q205: MMBT2222A, Package_TO_SOT_SMD:SOT-23-3, symbol Transistor_BJT:BC817
- added R204, R208: 100k, Resistor_SMD:R_0603_1608Metric_Pad0.98x0.95mm_HandSolder, symbol Device:R
- added R211: 511k, Resistor_SMD:R_0603_1608Metric_Pad0.98x0.95mm_HandSolder, symbol Device:R
- added R212: 91k, Resistor_SMD:R_0603_1608Metric_Pad0.98x0.95mm_HandSolder, symbol Device:R
- added SW201, SW203: SW_SPST, Connector_JST:JST_XH_B2B-XH-A_1x02_P2.50mm_Vertical, symbol Switch:SW_SPST
- added U204: TPS63802DLAR, TPS63802DLAR:VREG_TPS63802DLAR, symbol ECE477_PartsLibrary:TPS63802DLAR
- BT201: renamed from BT1; footprint (none) -> Connector_JST:JST_PH_S2B-PH-SM4-TB_1x02-1MP_P2.00mm_Horizontal; DigiKey Part (none) -> 455-S2B-PH-SM4-TBCT-ND
- C201: renamed from C5; footprint (none) -> Capacitor_SMD:C_0603_1608Metric_Pad1.08x0.95mm_HandSolder; DigiKey Part (none) -> 490-GRM188R60J106KE47JCT-ND
- C202: renamed from C8; footprint (none) -> Capacitor_SMD:C_0603_1608Metric_Pad1.08x0.95mm_HandSolder; DigiKey Part (none) -> 490-5405-1-ND
- C203: renamed from C14; value 10u -> 22uF; footprint (none) -> Capacitor_SMD:C_0603_1608Metric_Pad1.08x0.95mm_HandSolder; DigiKey Part (none) -> 490-7611-1-ND
- C204: renamed from C2; footprint (none) -> Capacitor_SMD:C_0603_1608Metric_Pad1.08x0.95mm_HandSolder; DigiKey Part (none) -> 490-7229-1-ND
- C205: renamed from C6; footprint (none) -> Capacitor_SMD:C_0603_1608Metric_Pad1.08x0.95mm_HandSolder; DigiKey Part (none) -> 490-GRM188R60J106KE47JCT-ND
- C206: renamed from C7; footprint (none) -> Capacitor_SMD:C_0603_1608Metric_Pad1.08x0.95mm_HandSolder; DigiKey Part (none) -> 490-GRM188R60J106KE47JCT-ND
- C207: renamed from C1; footprint (none) -> Capacitor_SMD:C_0603_1608Metric_Pad1.08x0.95mm_HandSolder; DigiKey Part (none) -> 445-5192-1-ND
- C209: renamed from C3; footprint (none) -> Capacitor_SMD:C_0603_1608Metric_Pad1.08x0.95mm_HandSolder; DigiKey Part (none) -> 490-GRM188R60J106KE47JCT-ND
- C210: renamed from C4; footprint (none) -> Capacitor_SMD:C_0603_1608Metric_Pad1.08x0.95mm_HandSolder; DigiKey Part (none) -> 490-7229-1-ND
- D201: renamed from D1; DigiKey Part (none) -> D5V0L1B2S9-7DICT-ND; LCSC Part Number C508181 -> (none)
- D202: renamed from D12; footprint Diode_SMD:D_0402_1005Metric_Pad0.77x0.64mm_HandSolder -> Diode_SMD:D_0805_2012Metric_Pad1.15x1.40mm_HandSolder; DigiKey Part (none) -> 475-LSR976-NR-1CT-ND; LCSC Part Number C136765 -> (none)
- D203: renamed from D2; DigiKey Part (none) -> D5V0L1B2S9-7DICT-ND; LCSC Part Number C508181 -> (none)
- D204: renamed from D13; footprint Diode_SMD:D_0402_1005Metric_Pad0.77x0.64mm_HandSolder -> Diode_SMD:D_0805_2012Metric_Pad1.15x1.40mm_HandSolder; DigiKey Part (none) -> 475-LSR976-NR-1CT-ND; LCSC Part Number C136765 -> (none)
- D205: renamed from D10; value PMEG40 -> PMEG4010BEA,115; DigiKey Part (none) -> 1727-5211-1-ND; LCSC Part Number C36975 -> (none)
- D209: renamed from D3; footprint (none) -> LED_SMD:LED_0805_2012Metric_Pad1.15x1.40mm_HandSolder; DigiKey Part (none) -> 475-LSR976-NR-1CT-ND
- D210: renamed from D4; footprint (none) -> LED_SMD:LED_0805_2012Metric_Pad1.15x1.40mm_HandSolder; DigiKey Part (none) -> 475-LSR976-NR-1CT-ND
- D211: renamed from D5; footprint (none) -> LED_SMD:LED_0805_2012Metric_Pad1.15x1.40mm_HandSolder; DigiKey Part (none) -> 475-LSR976-NR-1CT-ND
- J202: renamed from J2; footprint (none) -> Connector_PinHeader_2.54mm:PinHeader_1x02_P2.54mm_Vertical
- J203: renamed from J4; footprint (none) -> Connector_PinHeader_2.54mm:PinHeader_1x02_P2.54mm_Vertical
- Q202: renamed from Q1; value BC817 -> MMBT2222A; footprint Package_TO_SOT_SMD:SOT-23 -> Package_TO_SOT_SMD:SOT-23-3; DigiKey Part (none) -> 4878-MMBT2222ACT-ND
- R201: renamed from R7; footprint Resistor_SMD:R_0402_1005Metric_Pad0.72x0.64mm_HandSolder -> Resistor_SMD:R_0603_1608Metric_Pad0.98x0.95mm_HandSolder; DigiKey Part (none) -> 311-750GRCT-ND; LCSC Part Number C103153 -> (none)
- R202: renamed from R1; footprint Resistor_SMD:R_0402_1005Metric_Pad0.72x0.64mm_HandSolder -> Resistor_SMD:R_0603_1608Metric_Pad0.98x0.95mm_HandSolder; DigiKey Part (none) -> RMCF0603FT5K10CT-ND; LCSC Part Number C105872 -> (none)
- R203: renamed from R2; footprint Resistor_SMD:R_0402_1005Metric_Pad0.72x0.64mm_HandSolder -> Resistor_SMD:R_0603_1608Metric_Pad0.98x0.95mm_HandSolder; DigiKey Part (none) -> RMCF0603FT5K10CT-ND; LCSC Part Number C105872 -> (none)
- R205: renamed from R25; footprint (none) -> Resistor_SMD:R_0603_1608Metric_Pad0.98x0.95mm_HandSolder; DigiKey Part (none) -> 13-RC0603FR-13470RLCT-ND
- R206: renamed from R26; footprint (none) -> Resistor_SMD:R_0603_1608Metric_Pad0.98x0.95mm_HandSolder; DigiKey Part (none) -> RNCF0603TKY250RCT-ND
- R207: renamed from R3; footprint (none) -> Resistor_SMD:R_0603_1608Metric_Pad0.98x0.95mm_HandSolder; DigiKey Part (none) -> WSLJ-.01CT-ND
- R209: renamed from R18; value R -> 1k; footprint (none) -> Resistor_SMD:R_0603_1608Metric_Pad0.98x0.95mm_HandSolder; DigiKey Part (none) -> 311-1.00KHRCT-ND
- R210: renamed from R17; footprint (none) -> Resistor_SMD:R_0603_1608Metric_Pad0.98x0.95mm_HandSolder; DigiKey Part (none) -> 311-10KGRCT-ND
- R213: renamed from R19; footprint (none) -> Resistor_SMD:R_0603_1608Metric_Pad0.98x0.95mm_HandSolder; DigiKey Part (none) -> 311-10KGRCT-ND
- R214: renamed from R20; footprint (none) -> Resistor_SMD:R_0603_1608Metric_Pad0.98x0.95mm_HandSolder; DigiKey Part (none) -> 311-10KGRCT-ND
- R215: renamed from R8; footprint (none) -> Resistor_SMD:R_0603_1608Metric_Pad0.98x0.95mm_HandSolder; DigiKey Part (none) -> 311-1.00KHRCT-ND
- R216: renamed from R12; footprint (none) -> Resistor_SMD:R_0603_1608Metric_Pad0.98x0.95mm_HandSolder; DigiKey Part (none) -> 311-1.00KHRCT-ND
- R217: renamed from R13; footprint (none) -> Resistor_SMD:R_0603_1608Metric_Pad0.98x0.95mm_HandSolder; DigiKey Part (none) -> 311-1.00KHRCT-ND
- R218: renamed from R14; footprint (none) -> Resistor_SMD:R_0603_1608Metric_Pad0.98x0.95mm_HandSolder; DigiKey Part (none) -> 311-1.00KHRCT-ND
- R219: renamed from R15; footprint (none) -> Resistor_SMD:R_0603_1608Metric_Pad0.98x0.95mm_HandSolder; DigiKey Part (none) -> 311-1.00KHRCT-ND
- R220: renamed from R4; footprint (none) -> Resistor_SMD:R_0603_1608Metric_Pad0.98x0.95mm_HandSolder; DigiKey Part (none) -> 13-RC0603FR-13180RLCT-ND
- R221: renamed from R5; footprint (none) -> Resistor_SMD:R_0603_1608Metric_Pad0.98x0.95mm_HandSolder; DigiKey Part (none) -> 311-1.00KHRCT-ND
- R222: renamed from R6; footprint (none) -> Resistor_SMD:R_0603_1608Metric_Pad0.98x0.95mm_HandSolder; DigiKey Part (none) -> 311-750GRCT-ND
- R223: renamed from R9; footprint (none) -> Resistor_SMD:R_0603_1608Metric_Pad0.98x0.95mm_HandSolder; DigiKey Part (none) -> 311-10KGRCT-ND
- R224: renamed from R16; value 490 -> 590; footprint (none) -> Resistor_SMD:R_0603_1608Metric_Pad0.98x0.95mm_HandSolder; DigiKey Part (none) -> YAG3193CT-ND
- R225: renamed from R11; footprint (none) -> Resistor_SMD:R_0603_1608Metric_Pad0.98x0.95mm_HandSolder; DigiKey Part (none) -> 13-RC0603FR-131K5LCT-ND
- R226: renamed from R10; footprint (none) -> Resistor_SMD:R_0603_1608Metric_Pad0.98x0.95mm_HandSolder; DigiKey Part (none) -> 13-RC0603FR-1322RLCT-ND
- RN201: renamed from RN1; footprint (none) -> Resistor_SMD:R_Array_Convex_2x0606; DigiKey Part (none) -> Y8472CT-ND
- U201: renamed from U7; DigiKey Part (none) -> 296-LMS33460MGCT-ND
- U202: renamed from U3; DigiKey Part (none) -> 296-39461-1-ND
- U203: renamed from U2; DigiKey Part (none) -> 296-39941-1-ND
- U205: renamed from U1; value BQ24075RGT -> BQ24075RGTR; DigiKey Part (none) -> 296-38874-1-ND
Connections:
- net +3V3: now also JP203.2 (B), JP204.2 (B), Q201.3 (C)
- net +5V: now also C212.1, D206.2 (A2), FB201.2
- net BAT.EN1: now also Q203.1 (B)
- net BAT.EN2: now also Q204.1 (B)
- net BAT.OFF: now also R204.2, SW201.1 (A)
- net BAT.TMR: now also Q205.1 (B)
- net BAT.~{CE}: now also SW203.1 (A)
- net EN1: now also Q203.2 (E)
- net EN2: now also Q204.2 (E)
- net GND: now also C208.2, C211.2, C212.2, D206.1 (A1), J204.A1 (GND), J204.A12 (GND), J204.B1 (GND), J204.B12 (GND), J204.S1 (SHIELD), R204.1, R212.2, U204.2 (MODE), U204.3 (AGND), U204.8 (GND)
- net SYS.PWR: now also JP201.1 (A), JP202.1 (A), Q203.3 (C), Q204.3 (C), SW203.2 (B)
- net TMR: now also Q205.3 (C)
- net USB.D+: now also J204.A6 (D+), J204.B6 (D+)
- net USB.D-: now also J204.A7 (D-), J204.B7 (D-)
- net USB.Detect: now also Q201.2 (E)
- net V_BAT: now also SW201.2 (B)
- net V_RAW: now also C211.1, FB201.1, J204.A4 (VBUS), J204.A9 (VBUS), J204.B4 (VBUS), J204.B9 (VBUS)
- net at C201.1, U202.5 (VIN): now also JP201.2 (B)
- net at C205.1, C206.1, U202.1 (VOUT)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: now also JP203.1 (A)
- net at C203.1: now also JP202.2 (B), R208.1, U204.1 (EN), U204.10 (VIN)
- net at U202.2 (L2): now also L202.1
- net at U202.4 (L1): now also L202.2
- net at R203.2: now also J204.B5 (CC2)
- net at R202.1: now also J204.A5 (CC1)
- net at D205.1 (K): now also Q201.1 (B)
- net at R226.1: now also Q205.2 (E)
- new net: L203.1, U204.9 (L1)
- new net: L203.2, U204.7 (L2)
- new net: R211.2, R212.1, U204.4 (FB)
- new net: R208.2, U204.5 (PG)
- new net: C208.1, JP204.1 (A), R211.1, U204.6 (VOUT)
- no-connect marks 4 -> 2
Other:
- note added: "USB PWR Filtering"
- moved on the sheet: C201, C202, C203, C205, C206, D201, D202, D203, D204, R201, R205, R206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

Commit message: Update 90% done
Parts:
- removed BT201: Battery_Cell, Connector_JST:JST_PH_S2B-PH-SM4-TB_1x02-1MP_P2.00mm_Horizontal, symbol Device:Battery_Cell
- removed C201, C205: 10u, Capacitor_SMD:C_0603_1608Metric_Pad1.08x0.95mm_HandSolder, symbol Device:C
- removed C202: 0.1u, Capacitor_SMD:C_0603_1608Metric_Pad1.08x0.95mm_HandSolder, symbol Device:C
- removed L202: 1.5u, IND_TAIYO_NR3015_TAY, symbol ECE477_PartsLibrary:NR3015T1R5N
- removed U202: TPS63031DSK, Package_SON:WSON-10-1EP_2.5x2.5mm_P0.5mm_EP1.2x2mm, symbol Regulator_Switching:TPS63031DSK
- added C203: 10u, Capacitor_SMD:C_0603_1608Metric_Pad1.08x0.95mm_HandSolder, symbol Device:C
- added C208: 22u, Capacitor_SMD:C_0603_1608Metric_Pad1.08x0.95mm_HandSolder, symbol Device:C
- added D210: 3757-SS12L_R1_00001CT-ND, Diode_SMD:D_SMA, symbol Device:D_Schottky
- added J202: Conn_01x02_Pin, ECE477_PartsLibrary:CONN_S2B-PH-K-S_JST, symbol Connector:Conn_01x02_Pin
- added J206: Conn_01x10_Socket, ECE477_PartsLibrary:ECE477_BATBabySitter, symbol Connector:Conn_01x10_Socket
- added L201: 1u, ECE477_PartsLibrary:IND_XFL4020-102MEC, symbol ECE477_PartsLibrary:NR3015T1R5N
- added R209: 453k, Resistor_SMD:R_0603_1608Metric_Pad0.98x0.95mm_HandSolder, symbol Device:R
- added R210: 100k, Resistor_SMD:R_0603_1608Metric_Pad0.98x0.95mm_HandSolder, symbol Device:R
- added R215: 1M, Resistor_SMD:R_0603_1608Metric_Pad0.98x0.95mm_HandSolder, symbol Device:R
- added U202: TPS63021DSJR, ECE477_PartsLibrary:IC_TPS63021DSJR, symbol ECE477_PartsLibrary:TPS63021DSJR
- C201: renamed from C211; Manufacturer (none) -> Murata Electronics; Mfg. Part # (none) -> GRM033R61A104ME15D; Package (none) -> 0603; Supplier (none) -> DigiKey; Supplier Part # (none) -> 490-5405-1-ND
- C202: renamed from C212; Manufacturer (none) -> Murata Electronics; Mfg. Part # (none) -> GRM033R61A104ME15D; Package (none) -> 0603; Supplier (none) -> DigiKey; Supplier Part # (none) -> 490-5405-1-ND
- C204: renamed from C203; value 22uF -> 22u; Manufacturer (none) -> Murata Electronics; Mfg. Part # (none) -> GRM188R60J226MEA0D; Package (none) -> 0603; Supplier (none) -> DigiKey; Supplier Part # (none) -> 490-7611-1-ND
- C205: renamed from C204; Manufacturer (none) -> Murata Electronics; Mfg. Part # (none) -> GRM033R60J105MEA2D; Package (none) -> 0603; Supplier (none) -> DigiKey; Supplier Part # (none) -> 490-7229-1-ND
- C206: value 10u -> 22u; DigiKey Part 490-GRM188R60J106KE47JCT-ND -> 445-9077-1-ND; Manufacturer (none) -> TDK Corporation; Mfg. Part # (none) -> C1608X5R1A226M080AC; Package (none) -> 0603; Supplier (none) -> DigiKey; Supplier Part # (none) -> 445-9077-1-ND
- C207: Manufacturer (none) -> TDK Corporation; Mfg. Part # (none) -> C1608X7R1C474K080AC; Package (none) -> 0603; Supplier (none) -> DigiKey; Supplier Part # (none) -> 445-5192-1-ND
- C209: renamed from C208; Manufacturer (none) -> TDK Corporation; Mfg. Part # (none) -> C1608X5R1A226M080AC; Package (none) -> 0603; Supplier (none) -> DigiKey; Supplier Part # (none) -> 445-9077-1-ND
- C210: renamed from C209; Manufacturer (none) -> Murata Electronics; Mfg. Part # (none) -> GRM188R60J106KE47J; Package (none) -> 0603; Supplier (none) -> DigiKey; Supplier Part # (none) -> 490-GRM188R60J106KE47JCT-ND
- C211: renamed from C210; Manufacturer (none) -> Murata Electronics; Mfg. Part # (none) -> GRM033R60J105MEA2D; Package (none) -> 0603; Supplier (none) -> DigiKey; Supplier Part # (none) -> 490-7229-1-ND
- D201, D203: value D5V0L1B2S9-7 -> D5V0L1B2T-7; footprint Diode_SMD:D_SOD-923 -> Diode_SMD:D_SOD-523; DigiKey Part D5V0L1B2S9-7DICT-ND -> D5V0L1B2T-7DICT-ND; Manufacturer (none) -> Diodes Incorporated; Mfg. Part # (none) -> D5V0L1B2T-7; Package (none) -> SOD-523; Supplier (none) -> DigiKey; Supplier Part # (none) -> D5V0L1B2T-7DICT-ND
- D202: Manufacturer (none) -> ams-OSRAM USA INC.; Mfg. Part # (none) -> LS R976-NR-1; Package (none) -> 0805; Supplier (none) -> DigiKey; Supplier Part # (none) -> 475-LSR976-NR-1CT-ND
- D204: renamed from D206; value D5V0L1B2S9-7 -> D5V0L1B2T-7; footprint Diode_SMD:D_SOD-923 -> Diode_SMD:D_SOD-523; DigiKey Part D5V0L1B2S9-7DICT-ND -> D5V0L1B2T-7DICT-ND; Manufacturer (none) -> Diodes Incorporated; Mfg. Part # (none) -> D5V0L1B2T-7; Package (none) -> SOD-523; Supplier (none) -> DigiKey; Supplier Part # (none) -> D5V0L1B2T-7DICT-ND
- D205: renamed from D204; Manufacturer (none) -> ams-OSRAM USA INC.; Mfg. Part # (none) -> LS R976-NR-1; Package (none) -> 0805; Supplier (none) -> DigiKey; Supplier Part # (none) -> 475-LSR976-NR-1CT-ND
- D206: renamed from D205; value PMEG4010BEA,115 -> 3757-SS12L_R1_00001CT-ND; footprint Diode_SMD:D_SOD-323 -> Diode_SMD:D_SMA; DigiKey Part 1727-5211-1-ND -> 846-RBS2LAM40BCT-ND; Manufacturer (none) -> Panjit International Inc.; Mfg. Part # (none) -> SS12L_R1_00001; Package (none) -> SOD-128; Supplier (none) -> DigiKey; Supplier Part # (none) -> 3757-SS12L_R1_00001CT-ND
- D207: renamed from D209; Manufacturer (none) -> ams-OSRAM USA INC.; Mfg. Part # (none) -> LS R976-NR-1; Package (none) -> 0805; Supplier (none) -> DigiKey; Supplier Part # (none) -> 475-LSR976-NR-1CT-ND
- D208: renamed from D210; Manufacturer (none) -> ams-OSRAM USA INC.; Mfg. Part # (none) -> LS R976-NR-1; Package (none) -> 0805; Supplier (none) -> DigiKey; Supplier Part # (none) -> 475-LSR976-NR-1CT-ND
- D209: renamed from D211; Manufacturer (none) -> ams-OSRAM USA INC.; Mfg. Part # (none) -> LS R976-NR-1; Package (none) -> 0805; Supplier (none) -> DigiKey; Supplier Part # (none) -> 475-LSR976-NR-1CT-ND
- FB201: Manufacturer (none) -> Murata Electronics; Mfg. Part # (none) -> BLM18BD121SH1D; Package (none) -> 0603; Supplier (none) -> DigiKey; Supplier Part # (none) -> 490-17710-1-ND
- J201: renamed from J204; Manufacturer (none) -> GCT; Mfg. Part # (none) -> USB4105-GF-A; Package (none) -> USB2.0 TYP C 24P; Supplier (none) -> DigiKey; Supplier Part # (none) -> 2073-USB4105-GF-ACT-ND
- J203: renamed from J202; Supplier (none) -> Amazon
- J204: renamed from J203; Supplier (none) -> Amazon
- JP201, JP203: footprint (none) -> Jumper:SolderJumper-2_P1.3mm_Open_Pad1.0x1.5mm; Supplier (none) -> Amazon
- JP202, JP204: footprint (none) -> Jumper:SolderJumper-2_P1.3mm_Bridged_Pad1.0x1.5mm; Supplier (none) -> Amazon
- L202: renamed from L203; footprint IND_IHLP-2020CZ -> ECE477_PartsLibrary:IND_IHLP-2020CZ; Manufacturer (none) -> Vishay Dale; Mfg. Part # (none) -> IHLP2020CZERR47M11; Package (none) -> IHLP2020CZERR47M11; Supplier (none) -> DigiKey; Supplier Part # (none) -> 541-1231-1-ND
- Q201, Q202, Q203, Q204, Q205: Manufacturer (none) -> Diotec Semiconductor; Mfg. Part # (none) -> MMBT2222A; Package (none) -> SOT-23-3; Supplier (none) -> DigiKey; Supplier Part # (none) -> 4878-MMBT2222ACT-ND
- R201: renamed from R204; Manufacturer (none) -> YAGEO; Mfg. Part # (none) -> RC0603FR-07100KL; Package (none) -> 0603; Supplier (none) -> DigiKey; Supplier Part # (none) -> 311-100KHRCT-ND
- R202: renamed from R201; Manufacturer (none) -> YAGEO; Mfg. Part # (none) -> RC0603JR-07750RL; Package (none) -> 0603; Supplier (none) -> DigiKey; Supplier Part # (none) -> 311-750GRCT-ND
- R203: renamed from R202; Manufacturer (none) -> Stackpole Electronics Inc; Mfg. Part # (none) -> RMCF0603FT5K10; Package (none) -> 0603; Supplier (none) -> DigiKey; Supplier Part # (none) -> RMCF0603FT5K10CT-ND
- R204: renamed from R203; Manufacturer (none) -> Stackpole Electronics Inc; Mfg. Part # (none) -> RMCF0603FT5K10; Package (none) -> 0603; Supplier (none) -> DigiKey; Supplier Part # (none) -> RMCF0603FT5K10CT-ND
- R205: Manufacturer (none) -> YAGEO; Mfg. Part # (none) -> RC0603FR-13470RL; Package (none) -> 0603; Supplier (none) -> DigiKey; Supplier Part # (none) -> 13-RC0603FR-13470RLCT-ND
- R206: Manufacturer (none) -> Stackpole Electronics Inc; Mfg. Part # (none) -> RNCF0603TKY250R; Package (none) -> 0603; Supplier (none) -> DigiKey; Supplier Part # (none) -> RNCF0603TKY250RCT-ND
- R207: Manufacturer (none) -> Vishay Dale; Mfg. Part # (none) -> WSL0603R0100FEA; Package (none) -> 0603; Supplier (none) -> DigiKey; Supplier Part # (none) -> WSLJ-.01CT-ND
- R208: Manufacturer (none) -> YAGEO; Mfg. Part # (none) -> RC0603FR-07100KL; Package (none) -> 0603; Supplier (none) -> DigiKey; Supplier Part # (none) -> 311-100KHRCT-ND
- R211: renamed from R209; Manufacturer (none) -> YAGEO; Mfg. Part # (none) -> RC0603FR-071KL; Package (none) -> 0603; Supplier (none) -> DigiKey; Supplier Part # (none) -> 311-1.00KHRCT-ND
- R212: renamed from R210; Manufacturer (none) -> YAGEO; Mfg. Part # (none) -> RC0603JR-0710KL; Package (none) -> 0603; Supplier (none) -> DigiKey; Supplier Part # (none) -> 311-10KGRCT-ND
- R213: renamed from R211; Manufacturer (none) -> Vishay Dale; Mfg. Part # (none) -> CRCW0603511KFKEA; Package (none) -> 0603; Supplier (none) -> DigiKey; Supplier Part # (none) -> 541-511KHCT-ND
- R214: renamed from R212; Manufacturer (none) -> YAGEO; Mfg. Part # (none) -> RC0603FR-0791KL; Package (none) -> 0603; Supplier (none) -> DigiKey; Supplier Part # (none) -> 311-91.0KHRCT-ND
- R216: renamed from R213; Manufacturer (none) -> YAGEO; Mfg. Part # (none) -> RC0603JR-0710KL; Package (none) -> 0603; Supplier (none) -> DigiKey; Supplier Part # (none) -> 311-10KGRCT-ND
- R217: renamed from R214; Manufacturer (none) -> YAGEO; Mfg. Part # (none) -> RC0603JR-0710KL; Package (none) -> 0603; Supplier (none) -> DigiKey; Supplier Part # (none) -> 311-10KGRCT-ND
- R218: renamed from R215; Manufacturer (none) -> YAGEO; Mfg. Part # (none) -> RC0603FR-071KL; Package (none) -> 0603; Supplier (none) -> DigiKey; Supplier Part # (none) -> 311-1.00KHRCT-ND
- R219: renamed from R216; Manufacturer (none) -> YAGEO; Mfg. Part # (none) -> RC0603FR-071KL; Package (none) -> 0603; Supplier (none) -> DigiKey; Supplier Part # (none) -> 311-1.00KHRCT-ND
- R220: renamed from R217; Manufacturer (none) -> YAGEO; Mfg. Part # (none) -> RC0603FR-071KL; Package (none) -> 0603; Supplier (none) -> DigiKey; Supplier Part # (none) -> 311-1.00KHRCT-ND
- R221: renamed from R218; Manufacturer (none) -> YAGEO; Mfg. Part # (none) -> RC0603FR-071KL; Package (none) -> 0603; Supplier (none) -> DigiKey; Supplier Part # (none) -> 311-1.00KHRCT-ND
- R222: renamed from R219; Manufacturer (none) -> YAGEO; Mfg. Part # (none) -> RC0603FR-071KL; Package (none) -> 0603; Supplier (none) -> DigiKey; Supplier Part # (none) -> 311-1.00KHRCT-ND
- R223: renamed from R220; Manufacturer (none) -> YAGEO; Mfg. Part # (none) -> RC0603FR-13180RL; Package (none) -> 0603; Supplier (none) -> DigiKey; Supplier Part # (none) -> 13-RC0603FR-13180RLCT-ND
- R224: renamed from R221; Manufacturer (none) -> YAGEO; Mfg. Part # (none) -> RC0603FR-071KL; Package (none) -> 0603; Supplier (none) -> DigiKey; Supplier Part # (none) -> 311-1.00KHRCT-ND
- R225: renamed from R222; Manufacturer (none) -> YAGEO; Mfg. Part # (none) -> RC0603JR-07750RL; Package (none) -> 0603; Supplier (none) -> DigiKey; Supplier Part # (none) -> 311-750GRCT-ND
- R226: renamed from R223; Manufacturer (none) -> YAGEO; Mfg. Part # (none) -> RC0603JR-0710KL; Package (none) -> 0603; Supplier (none) -> DigiKey; Supplier Part # (none) -> 311-10KGRCT-ND
- R227: renamed from R224; Manufacturer (none) -> YAGEO; Mfg. Part # (none) -> RC0402FR-07590RL; Package (none) -> 0603; Supplier (none) -> DigiKey; Supplier Part # (none) -> YAG3193CT-ND
- R228: renamed from R225; Manufacturer (none) -> YAGEO; Mfg. Part # (none) -> RC0603FR-131K5L; Package (none) -> 0603; Supplier (none) -> DigiKey; Supplier Part # (none) -> 13-RC0603FR-131K5LCT-ND
- R229: renamed from R226; Manufacturer (none) -> YAGEO; Mfg. Part # (none) -> RC0603FR-1322RL; Package (none) -> 0603; Supplier (none) -> DigiKey; Supplier Part # (none) -> 13-RC0603FR-1322RLCT-ND
- RN201: Manufacturer (none) -> Panasonic Electronic Components; Mfg. Part # (none) -> EXB-34V472JV; Package (none) -> 2x0606_Convex; Supplier (none) -> DigiKey; Supplier Part # (none) -> Y8472CT-ND
- SW201: Manufacturer (none) -> JST Sales America Inc.; Mfg. Part # (none) -> B2B-XH-A; Package (none) -> B2B-XH-A; Supplier (none) -> DigiKey; Supplier Part # (none) -> 455-B2B-XH-A-ND
- SW202: renamed from SW203; Manufacturer (none) -> JST Sales America Inc.; Mfg. Part # (none) -> B2B-XH-A; Package (none) -> B2B-XH-A; Supplier (none) -> DigiKey; Supplier Part # (none) -> 455-B2B-XH-A-ND
- U201: footprint LMS33460MG:SOT65P210X110-5N -> ECE477_PartsLibrary:SOT65P210X110-5N; Manufacturer (none) -> Texas Instruments; Mfg. Part # (none) -> LMS33460MG; Package (none) -> SOT-353; Supplier (none) -> DigiKey; Supplier Part # (none) -> 296-LMS33460MGCT-ND
- U203: Manufacturer (none) -> Texas Instruments; Mfg. Part # (none) -> BQ27441DRZR-G1A; Package (none) -> 12-VFDFN Exposed Pad; Supplier (none) -> DigiKey; Supplier Part # (none) -> 296-39941-1-ND
- U204: footprint TPS63802DLAR:VREG_TPS63802DLAR -> ECE477_PartsLibrary:VREG_TPS63802DLAR; Manufacturer (none) -> Texas Instruments; Mfg. Part # (none) -> TPS63802DLAR; Package (none) -> 10-VFDFN; Supplier (none) -> DigiKey; Supplier Part # (none) -> 296-TPS63802DLARCT-ND
- U205: footprint Package_DFN_QFN:VQFN-16-1EP_3x3mm_P0.5mm_EP1.6x1.6mm -> Package_DFN_QFN:VQFN-16-1EP_3x3mm_P0.5mm_EP1.6x1.6mm_ThermalVias; Manufacturer (none) -> Texas Instruments; Mfg. Part # (none) -> BQ24075RGTR; Package (none) -> 16-VFQFN Exposed Pad; Supplier (none) -> DigiKey; Supplier Part # (none) -> 296-38874-1-ND
Connections:
- net +3V3: now also J206.2 (Pin_2)
- net +5V: now also J206.9 (Pin_9)
- net BAT.GPOUT: now also J206.5 (Pin_5)
- net GND: now also C203.2, C208.2, J202.2 (Pin_2), J206.1 (Pin_1), J206.10 (Pin_10), J206.8 (Pin_8), R210.2, U202.1 (VINA), U202.12 (EN), U202.13 (PS/SYNC), U202.15 (PGND), U202.16 (PGND), U202.17 (PGND), U202.18 (PGND), U202.19 (PGND), U202.2 (GND), U202.20 (PGND), U202.21 (PGND), U202.22 (PGND), U202.23 (PGND), U202.24 (PGND), U202.25 (PGND), U202.26 (PGND), U202.27 (PGND), U202.28 (PGND), U202.29 (PGND), U202.30 (PGND)
- net I2C.SCL: now also J206.4 (Pin_4)
- net I2C.SDA: now also J206.3 (Pin_3)
- net SYS.PWR: now also J206.7 (Pin_7)
- net V_RAW: now also D210.2 (A); no longer FB201.1
- net ~{CE}: now also J206.6 (Pin_6)
- net at JP201.2 (B): now also C203.1, U202.10 (VIN), U202.11 (VIN)
- net at C206.1, JP203.1 (A): now also C208.1, R209.1, R215.1, U202.4 (VOUT), U202.5 (VOUT)
- net at C205.2, R207.2, U203.6 (BAT)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: now also J202.1 (Pin_1)
- net PWR_JP: now reaches C204.1, JP202.2 (B), R208.1, U204.1 (EN), U204.10 (VIN)
- net 3V_JP: now reaches C209.1, JP204.1 (A), R213.1, U204.6 (VOUT)
- new net: D210.1 (K), FB201.1
- new net: R209.2, R210.1, U202.3 (FB)
- new net: R215.2, U202.14 (PG)
- new net: L201.1, U202.6 (L2_6), U202.7 (L2_7)
- new net: L201.2, U202.8 (L1_8), U202.9 (L1_9)
- no-connect marks 2 -> 3
Other:
- moved on the sheet: C201, C202, D202, D204, D205, D206, FB201, Q201, R201, R202, R205, R206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

Commit message: design 02/17
Parts:
- removed J201: USB_C_Receptacle_USB2.0_16P, Connector_USB:USB_C_Receptacle_HRO_TYPE-C-31-M-12, symbol Connector:USB_C_Receptacle_USB2.0_16P
- removed R203, R204: 5.1k, Resistor_SMD:R_0603_1608Metric_Pad0.98x0.95mm_HandSolder, symbol Device:R
- added H201, H202, H203, H204: MountingHole, MountingHole:MountingHole_3.2mm_M3, symbol Mechanical:MountingHole
- added J201: USB Micro Receptacle, ECE477_PartsLibrary:AMPHENOL_10118192-0002LF, symbol ECE477_PartsLibrary:USB3076-XX-X_REVC5
- added J205: Conn_01x04_Pin, Connector_PinHeader_2.54mm:PinHeader_1x04_P2.54mm_Vertical, symbol Connector:Conn_01x04_Pin
- added TP201, TP202, TP203, TP205: TestPoint, TestPoint:TestPoint_Pad_D2.0mm, symbol Connector:TestPoint
- U202: Manufacturer (none) -> Texas Instruments; Mfg. Part # (none) -> TPS63021DSJR; Package (none) -> 14-VFDFN Exposed Pad; Supplier Amazon -> DigiKey; Supplier Part # (none) -> 296-27259-1-ND
Connections:
- net +3V3: now also TP203.1
- net +5V: now also TP201.1
- net GND: now also J201.5 (GND), J201.6 (SHIELD), J205.4 (Pin_4), TP202.1; no longer U202.17 (PGND), U202.18 (PGND), U202.19 (PGND), U202.20 (PGND), U202.21 (PGND), U202.22 (PGND), U202.23 (PGND), U202.24 (PGND), U202.25 (PGND), U202.26 (PGND), U202.27 (PGND), U202.28 (PGND), U202.29 (PGND), U202.30 (PGND)
- net SYS.PWR: now also TP205.1
- net USB.D+: now also J201.3 (D+), J205.2 (Pin_2)
- net USB.D-: now also J201.2 (D-), J205.3 (Pin_3)
- net V_RAW: now also J201.1 (VBUS), J205.1 (Pin_1)
- no-connect marks 3 -> 2

Commit message: Update Rev 2
Parts:
- removed J203, J204: Conn_01x02_Pin, Connector_PinHeader_2.54mm:PinHeader_1x02_P2.54mm_Vertical, symbol Connector:Conn_01x02_Pin
- removed Q203, Q204, Q205: MMBT2222A, Package_TO_SOT_SMD:SOT-23-3, symbol Transistor_BJT:BC817
- removed R220, R222: 1k, Resistor_SMD:R_0603_1608Metric_Pad0.98x0.95mm_HandSolder, symbol Device:R
- added S201: DS04-254-2-02BK-SMT, ECE477_PartsLibrary:SW_DS04-254-2-02BK-SMT, symbol ECE477_PartsLibrary:DS04-254-2-02BK-SMT
- J205: value Conn_01x04_Pin -> Conn_01x10_Pin
- R219, R221: value 1k -> 10k; DigiKey Part 311-1.00KHRCT-ND -> 311-10KGRCT-ND; Mfg. Part # RC0603FR-071KL -> RC0603JR-0710KL; Supplier Part # 311-1.00KHRCT-ND -> 311-10KGRCT-ND
Connections:
- net EN1: now also S201.2B
- net EN2: now also R221.2, S201.1B; no longer R221.1
- net GND: now also S201.1A, S201.2A; no longer R219.2, R221.2
- net SYS.PWR: now also R219.2, R221.1
- net TMR: now also R229.1
Other:
- company: (none) -> ECE477 - Team 4: KayO
- title: (none) -> Power Supply Units
