File: PCB/PSU.kicad_sch (KiCad schematic)
At the start: 76 parts, among them J201 USB Micro Receptacle, J202 Conn_01x02_Pin, J205 Conn_01x10_Pin, J206 Conn_01x10_Socket, Q201 MMBT2222A, Q202 MMBT2222A, SW201 SW_SPST, SW202 SW_SPST, U201 LMS33460MG, U202 TPS63021DSJR, U203 BQ27441DRZR-G1A, U204 TPS63802DLAR, U205 BQ24075RGTR

Commit message: Redesign bluetooth of v2
Parts:
- removed C208: 22u, Capacitor_SMD:C_0603_1608Metric_Pad1.08x0.95mm_HandSolder, symbol Device:C
- removed L201: 1u, ECE477_PartsLibrary:IND_XFL4020-102MEC, symbol ECE477_PartsLibrary:NR3015T1R5N
- removed R209: 453k, Resistor_SMD:R_0603_1608Metric_Pad0.98x0.95mm_HandSolder, symbol Device:R
- removed R210: 100k, Resistor_SMD:R_0603_1608Metric_Pad0.98x0.95mm_HandSolder, symbol Device:R
- removed R215: 1M, Resistor_SMD:R_0603_1608Metric_Pad0.98x0.95mm_HandSolder, symbol Device:R
- removed U202: TPS63021DSJR, ECE477_PartsLibrary:IC_TPS63021DSJR, symbol ECE477_PartsLibrary:TPS63021DSJR
- added J203: Conn_01x02_Pin, Connector_JST:JST_XH_B2B-XH-A_1x02_P2.50mm_Vertical, symbol Connector:Conn_01x02_Pin
- added U206: AP7363-33D-13, ECE477_PartsLibrary:TO252-3L_DIO, symbol Regulator_Linear:AP7361C-10E
- C201, C202, C203, C204, C205, C207, C209, C210, C211, FB201, R201, R202, R205, R206, R207, R208, R211, R212, R213, R214, R216, R217, R218, R219, R221, R223, R224, R225, R226, R227, R228, R229: Package 0603 -> (none)
- C206: value 22u -> 10u; DigiKey Part 445-9077-1-ND -> 445-9015-1-ND; Mfg. Part # C1608X5R1A226M080AC -> C1608X5R1E106M080AC; Package 0603 -> (none); Supplier Part # 445-9077-1-ND -> 445-9015-1-ND
- D201, D203, D204: Package SOD-523 -> (none)
- D202: footprint Diode_SMD:D_0805_2012Metric_Pad1.15x1.40mm_HandSolder -> LED_SMD:LED_0805_2012Metric_Pad1.15x1.40mm_HandSolder; Manufacturer ams-OSRAM USA INC. -> Würth Elektronik; Mfg. Part # LS R976-NR-1 -> 150080YS75000; Package 0805 -> (none); Supplier Part # 475-LSR976-NR-1CT-ND -> 732-4987-1-ND
- D205: footprint Diode_SMD:D_0805_2012Metric_Pad1.15x1.40mm_HandSolder -> LED_SMD:LED_0805_2012Metric_Pad1.15x1.40mm_HandSolder; Manufacturer ams-OSRAM USA INC. -> Würth Elektronik; Mfg. Part # LS R976-NR-1 -> 150080YS75000; Package 0805 -> (none); Supplier Part # 475-LSR976-NR-1CT-ND -> 732-4984-1-ND
- D206, D210: Package SOD-128 -> (none)
- D207, D208: Manufacturer ams-OSRAM USA INC. -> Würth Elektronik; Mfg. Part # LS R976-NR-1 -> 150080VS75000; Package 0805 -> (none); Supplier Part # 475-LSR976-NR-1CT-ND -> 732-4986-1-ND
- D209: Manufacturer ams-OSRAM USA INC. -> Würth Elektronik; Mfg. Part # LS R976-NR-1 -> 150080YS75000; Package 0805 -> (none); Supplier Part # 475-LSR976-NR-1CT-ND -> 732-4987-1-ND
- H201, H202, H203, H204, TP201, TP202, TP203, TP205: Supplier (none) -> N/A
- J201: Package USB Micro -> (none)
- J202: Package S2B-PH-K-S -> (none)
- J205, JP201, JP202, JP203, JP204: Supplier Amazon -> N/A
- J206: Package N/A -> (none)
- L202: Package IHLP2020CZERR47M11 -> (none)
- Q201, Q202: Package SOT-23-3 -> (none)
- RN201: Package 2x0606_Convex -> (none)
- S201: MANUFACTURER CUI Inc. -> (none); MAXIMUM_PACKAGE_HEIGHT 4.86 mm -> (none); PARTREV V0.0 -> (none); Package 0.1'' switch -> (none); STANDARD Manufacturer Recommendations -> (none)
- SW201, SW202: value SW_SPST -> SW_Push; Package B2B-XH-A -> (none)
- U201: Package SOT-353 -> (none)
- U203: Package 12-VFDFN Exposed Pad -> (none)
- U204: Package 10-VFDFN -> (none)
- U205: Package 16-VFQFN Exposed Pad -> (none)
Connections:
- net GND: now also J203.2 (Pin_2), U206.2 (GND)
- net at C205.2, J202.1 (Pin_1), R207.2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: now also J203.1 (Pin_1)
- net at C206.1, JP203.1 (A): now also U206.3 (VO)
- net at C203.1, JP201.2 (B): now also U206.1 (VI)
Other:
- note added: "Micro USB"
- note removed: "USB_C"
- moved on the sheet: C203, JP201, JP203

Commit message: Update PCB Design v2
Parts:
- C201, C202: footprint Capacitor_SMD:C_0603_1608Metric_Pad1.08x0.95mm_HandSolder -> Capacitor_SMD:C_0805_2012Metric_Pad1.18x1.45mm_HandSolder; Manufacturer Murata Electronics -> Samsung Electro-Mechanics; Mfg. Part # GRM033R61A104ME15D -> CL21B104KBCNNNC; Supplier Part # 490-5405-1-ND -> 1276-1003-1-ND
- C203, C206: footprint Capacitor_SMD:C_0603_1608Metric_Pad1.08x0.95mm_HandSolder -> Capacitor_SMD:C_0805_2012Metric_Pad1.18x1.45mm_HandSolder; Manufacturer TDK Corporation -> Samsung Electro-Mechanics; Mfg. Part # C1608X5R1E106M080AC -> CL21A106KOQNNNE; Supplier Part # 445-9015-1-ND -> 1276-1096-1-ND
- C204: footprint Capacitor_SMD:C_0603_1608Metric_Pad1.08x0.95mm_HandSolder -> Capacitor_SMD:C_0805_2012Metric_Pad1.18x1.45mm_HandSolder; Manufacturer Murata Electronics -> Samsung Electro-Mechanics; Mfg. Part # GRM188R60J226MEA0D -> CL21A226MPQNNNE; Supplier Part # 490-7611-1-ND -> 1276-2910-1-ND
- C205, C211: footprint Capacitor_SMD:C_0603_1608Metric_Pad1.08x0.95mm_HandSolder -> Capacitor_SMD:C_0805_2012Metric_Pad1.18x1.45mm_HandSolder; Manufacturer Murata Electronics -> Samsung Electro-Mechanics; Mfg. Part # GRM033R60J105MEA2D -> CL21B105KAFNNNE; Supplier Part # 490-7229-1-ND -> 1276-1066-1-ND
- C207: footprint Capacitor_SMD:C_0603_1608Metric_Pad1.08x0.95mm_HandSolder -> Capacitor_SMD:C_0805_2012Metric_Pad1.18x1.45mm_HandSolder; Manufacturer TDK Corporation -> Samsung Electro-Mechanics; Mfg. Part # C1608X7R1C474K080AC -> CL21B474KBFNNNG; Supplier Part # 445-5192-1-ND -> 1276-6482-1-ND
- C209: footprint Capacitor_SMD:C_0603_1608Metric_Pad1.08x0.95mm_HandSolder -> Capacitor_SMD:C_0805_2012Metric_Pad1.18x1.45mm_HandSolder; Manufacturer TDK Corporation -> Samsung Electro-Mechanics; Mfg. Part # C1608X5R1A226M080AC -> CL21A226MPQNNNE; Supplier Part # 445-9077-1-ND -> 1276-2910-1-ND
- C210: footprint Capacitor_SMD:C_0603_1608Metric_Pad1.08x0.95mm_HandSolder -> Capacitor_SMD:C_0805_2012Metric_Pad1.18x1.45mm_HandSolder; Manufacturer Murata Electronics -> Samsung Electro-Mechanics; Mfg. Part # GRM188R60J106KE47J -> CL21A106KOQNNNE; Supplier Part # 490-GRM188R60J106KE47JCT-ND -> 1276-1096-1-ND
- J206, JP202, JP204: now left out of the parts list
- R201, R208: footprint Resistor_SMD:R_0603_1608Metric_Pad0.98x0.95mm_HandSolder -> Resistor_SMD:R_0805_2012Metric_Pad1.20x1.40mm_HandSolder; Mfg. Part # RC0603FR-07100KL -> RC0805FR-07100KL; Supplier Part # 311-100KHRCT-ND -> 311-100KCRCT-ND
- R202, R225: footprint Resistor_SMD:R_0603_1608Metric_Pad0.98x0.95mm_HandSolder -> Resistor_SMD:R_0805_2012Metric_Pad1.20x1.40mm_HandSolder; Mfg. Part # RC0603JR-07750RL -> RC0805FR-07750RL; Supplier Part # 311-750GRCT-ND -> 311-750CRCT-ND
- R205: footprint Resistor_SMD:R_0603_1608Metric_Pad0.98x0.95mm_HandSolder -> Resistor_SMD:R_0805_2012Metric_Pad1.20x1.40mm_HandSolder; Mfg. Part # RC0603FR-13470RL -> RC0805FR-07470RL; Supplier Part # 13-RC0603FR-13470RLCT-ND -> 311-470CRCT-ND
- R206: value 250 -> 330; footprint Resistor_SMD:R_0603_1608Metric_Pad0.98x0.95mm_HandSolder -> Resistor_SMD:R_0805_2012Metric_Pad1.20x1.40mm_HandSolder; Manufacturer Stackpole Electronics Inc -> YAGEO; Mfg. Part # RNCF0603TKY250R -> RC0805FR-07330RL; Supplier Part # RNCF0603TKY250RCT-ND -> 311-330CRCT-ND
- R207: footprint Resistor_SMD:R_0603_1608Metric_Pad0.98x0.95mm_HandSolder -> ECE477_PartsLibrary:RES_2012_SUS; Manufacturer Vishay Dale -> Susumu; Mfg. Part # WSL0603R0100FEA -> KRL2012E-M-R010-F-T5; Supplier Part # WSLJ-.01CT-ND -> 408-1600-1-ND
- R211, R218, R224: footprint Resistor_SMD:R_0603_1608Metric_Pad0.98x0.95mm_HandSolder -> Resistor_SMD:R_0805_2012Metric_Pad1.20x1.40mm_HandSolder; Mfg. Part # RC0603FR-071KL -> RC0805FR-071KL; Supplier Part # 311-1.00KHRCT-ND -> 311-1.00KCRCT-ND
- R212, R216, R217, R219, R221, R226: footprint Resistor_SMD:R_0603_1608Metric_Pad0.98x0.95mm_HandSolder -> Resistor_SMD:R_0805_2012Metric_Pad1.20x1.40mm_HandSolder; Mfg. Part # RC0603JR-0710KL -> RC0805FR-0710KL; Supplier Part # 311-10KGRCT-ND -> 311-10.0KCRCT-ND
- R213: footprint Resistor_SMD:R_0603_1608Metric_Pad0.98x0.95mm_HandSolder -> Resistor_SMD:R_0805_2012Metric_Pad1.20x1.40mm_HandSolder; Manufacturer Vishay Dale -> YAGEO; Mfg. Part # CRCW0603511KFKEA -> RC0805FR-07511KL; Supplier Part # 541-511KHCT-ND -> 311-511KCRCT-ND
- R214: footprint Resistor_SMD:R_0603_1608Metric_Pad0.98x0.95mm_HandSolder -> Resistor_SMD:R_0805_2012Metric_Pad1.20x1.40mm_HandSolder; Mfg. Part # RC0603FR-0791KL -> RC0805FR-0791KL; Supplier Part # 311-91.0KHRCT-ND -> 311-91.0KCRCT-ND
- R223: footprint Resistor_SMD:R_0603_1608Metric_Pad0.98x0.95mm_HandSolder -> Resistor_SMD:R_0805_2012Metric_Pad1.20x1.40mm_HandSolder; Mfg. Part # RC0603FR-13180RL -> RC0805JR-07180RL; Supplier Part # 13-RC0603FR-13180RLCT-ND -> 311-180ARCT-ND
- R227: footprint Resistor_SMD:R_0603_1608Metric_Pad0.98x0.95mm_HandSolder -> Resistor_SMD:R_0805_2012Metric_Pad1.20x1.40mm_HandSolder; Mfg. Part # RC0402FR-07590RL -> RC0805FR-07590RL; Supplier Part # YAG3193CT-ND -> 311-590CRCT-ND
- R228: footprint Resistor_SMD:R_0603_1608Metric_Pad0.98x0.95mm_HandSolder -> Resistor_SMD:R_0805_2012Metric_Pad1.20x1.40mm_HandSolder; Mfg. Part # RC0603FR-131K5L -> RC0805FR-071K5L; Supplier Part # 13-RC0603FR-131K5LCT-ND -> 311-1.50KCRCT-ND
- R229: footprint Resistor_SMD:R_0603_1608Metric_Pad0.98x0.95mm_HandSolder -> Resistor_SMD:R_0805_2012Metric_Pad1.20x1.40mm_HandSolder; Mfg. Part # RC0603FR-1322RL -> RC0805JR-0722RL; Supplier Part # 13-RC0603FR-1322RLCT-ND -> 311-22ARCT-ND

Commit message: PCB Update
Parts:
- D201, D203, D204: value D5V0L1B2T-7 -> D5V0L1B2WS-7; footprint Diode_SMD:D_SOD-523 -> Diode_SMD:D_SOD-323_HandSoldering; Mfg. Part # D5V0L1B2T-7 -> D5V0L1B2WS-7; Supplier Part # D5V0L1B2T-7DICT-ND -> D5V0L1B2WS-7DICT-ND
Changed lines of the file:
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@@
       (effects (font (size 1.27 1.27)) (justify left))
     )
-    (property "Value" "D5V0L1B2T-7" (at 67.945 144.7801 90)
-      (effects (font (size 1.27 1.27)) (justify left))
-    )
-    (property "Footprint" "Diode_SMD:D_SOD-523" (at 66.04 135.89 0)
+    (property "Value" "D5V0L1B2WS-7" (at 67.945 144.7801 90)
+      (effects (font (size 1.27 1.27)) (justify left))
+    )
+    (property "Footprint" "Diode_SMD:D_SOD-323_HandSoldering" (at 66.04 135.89 0)
       (effects (font (size 1.27 1.27)) hide)
     )
@@
       (effects (font (size 1.27 1.27)) hide)
     )
-    (property "Mfg. Part #" "D5V0L1B2T-7" (at 66.04 135.89 0)
+    (property "Mfg. Part #" "D5V0L1B2WS-7" (at 66.04 135.89 0)
       (effects (font (size 1.27 1.27)) hide)
     )
@@
       (effects (font (size 1.27 1.27)) hide)
     )
-    (property "Supplier Part #" "D5V0L1B2T-7DICT-ND" (at 66.04 135.89 0)
+    (property "Supplier Part #" "D5V0L1B2WS-7DICT-ND" (at 66.04 135.89 0)
       (effects (font (size 1.27 1.27)) hide)
     )
@@
       (effects (font (size 1.27 1.27)) (justify right))
     )
-    (property "Value" "D5V0L1B2T-7" (at 48.895 66.04 90)
+    (property "Value" "D5V0L1B2WS-7" (at 48.895 66.04 90)
       (effects (font (size 1.27 1.27)) (justify right))
     )
-    (property "Footprint" "Diode_SMD:D_SOD-523" (at 50.8 64.77 0)
+    (property "Footprint" "Diode_SMD:D_SOD-323_HandSoldering" (at 50.8 64.77 0)
       (effects (font (size 1.27 1.27)) hide)
     )
@@
       (effects (font (size 1.27 1.27)) hide)
     )
-    (property "Mfg. Part #" "D5V0L1B2T-7" (at 50.8 64.77 0)
+    (property "Mfg. Part #" "D5V0L1B2WS-7" (at 50.8 64.77 0)
       (effects (font (size 1.27 1.27)) hide)
     )
@@
       (effects (font (size 1.27 1.27)) hide)
     )
-    (property "Supplier Part #" "D5V0L1B2T-7DICT-ND" (at 50.8 64.77 0)
+    (property "Supplier Part #" "D5V0L1B2WS-7DICT-ND" (at 50.8 64.77 0)
       (effects (font (size 1.27 1.27)) hide)
     )
@@
       (effects (font (size 1.27 1.27)) (justify right))
     )
-    (property "Value" "D5V0L1B2T-7" (at 57.785 59.69 90)
+    (property "Value" "D5V0L1B2WS-7" (at 57.785 59.69 90)
       (effects (font (size 1.27 1.27)) (justify right))
     )
-    (property "Footprint" "Diode_SMD:D_SOD-523" (at 55.88 58.42 0)
+    (property "Footprint" "Diode_SMD:D_SOD-323_HandSoldering" (at 55.88 58.42 0)
       (effects (font (size 1.27 1.27)) hide)
     )
@@
       (effects (font (size 1.27 1.27)) hide)
     )
-    (property "Mfg. Part #" "D5V0L1B2T-7" (at 55.88 58.42 0)
+    (property "Mfg. Part #" "D5V0L1B2WS-7" (at 55.88 58.42 0)
       (effects (font (size 1.27 1.27)) hide)
     )
@@
       (effects (font (size 1.27 1.27)) hide)
     )
-    (property "Supplier Part #" "D5V0L1B2T-7DICT-ND" (at 55.88 58.42 0)
-      (effects (font (size 1.27 1.27)) hide)
-    )
+    (property "Supplier Part #" "D5V0L1B2WS-7DICT-ND" (at 55.88 58.42 0)
+      (effects (font (size 1.27 1.27)) hide)
+    )
