File: PCB/peri.kicad_sch (KiCad schematic)
At the start: 3 parts, among them J1 Micro_SD_Card, U4 RN42

Commit message: PCB init - Minh
Parts:
- added J6: BT SPI Debug, symbol Connector:Conn_01x06_Pin
Connections:
- net GND: now reaches U4.1 (GND)
- net GND: now also U4.12 (GND), U4.28 (GND), U4.29 (GND), U4.36 (SHIELD), J6.6 (Pin_6)
- net +3V3: now reaches U4.11 (VDD)
- net +3V3: now also J6.5 (Pin_5)
- net BT.RX: now reaches U4.13 (UART_RX)
- net BT.TX: now reaches U4.14 (UART_TX)
- net BT.RTS: now reaches U4.15 (UART_RTS)
- net BT.CTS: now reaches U4.16 (UART_CTS)
- net BT.MOSI: now reaches U4.2 (SPI_MOSI)
- net BT.MOSI: now also J6.2 (Pin_2)
- net BT.~{CS}: now reaches U4.23 (SPI_CSB)
- net BT.~{CS}: now also J6.4 (Pin_4)
- net BT.MISO: now reaches U4.24 (SPI_MISO)
- net BT.MISO: now also J6.3 (Pin_3)
- net BT.~{RST}: now reaches U4.5 (RESET)
- net BT.SCLK: now reaches U4.6 (SPI_CLK)
- net BT.SCLK: now also J6.1 (Pin_1)
- no-connect marks 0 -> 6
Other:
- moved on the sheet: J1, U4

Commit message: PCB update - Minh
Parts:
- J6: value BT SPI Debug -> SPI Debug
Connections:
- net +3V3: now also J1.4 (VDD)
- net BT.MISO: no longer U4.24 (SPI_MISO)
- net BT.MOSI: no longer U4.2 (SPI_MOSI)
- net BT.SCLK: no longer U4.6 (SPI_CLK)
- net BT.~{CS}: no longer U4.23 (SPI_CSB)
- net GND: now also J1.6 (VSS)
- net SPI.~{CS}: now reaches J1.2 (DAT3/CD)
- net SPI.~{CS}: now also U4.23 (SPI_CSB)
- net SPI.MOSI: now reaches J1.3 (CMD)
- net SPI.MOSI: now also U4.2 (SPI_MOSI)
- net SPI.SCLK: now reaches J1.5 (CLK)
- net SPI.SCLK: now also U4.6 (SPI_CLK)
- net SPI.MISO: now reaches J1.7 (DAT0)
- net SPI.MISO: now also U4.24 (SPI_MISO)
- no-connect marks 6 -> 8
Other:
- moved on the sheet: J6

Commit message: PCB update - Minh
Parts:
- removed DS1: OLED-128O064D, Display:OLED-128O064D, symbol Display_Graphic:OLED-128O064D
- added J5: BT USB Debug, symbol Connector:Conn_01x04_Pin
- added J7: UART Debug, symbol Connector:Conn_01x06_Pin
- added U8: 362 TFT LCD, symbol ECE477_PartsLibrary:362_OLED
Connections:
- net BT.MISO is gone; now on net SPI.MISO: J6.3 (Pin_3)
- net BT.MOSI is gone; now on net SPI.MOSI: J6.2 (Pin_2)
- net BT.SCLK is gone; now on net SPI.SCLK: J6.1 (Pin_1)
- net BT.~{CS} is gone; now on net SPI.~{CS}: J6.4 (Pin_4)
- net +3V3: now also J7.5 (Pin_5), U8.1 (VCC)
- net BT.CTS: now also J7.3 (Pin_3)
- net BT.RTS: now also J7.4 (Pin_4)
- net BT.RX: now also J7.2 (Pin_2)
- net BT.TX: now also J7.1 (Pin_1)
- net GND: now also J5.4 (Pin_4), J7.6 (Pin_6), U8.2 (GND)
- net SPI.MISO: now also U8.6 (SDO/MISO)
- net SPI.MOSI: now also U8.9 (SDI/MOSI)
- net SPI.SCLK: now also U8.7 (SCK)
- net SPI.~{CS}: now also U8.3 (CS)
- net BT.D+: now reaches U4.17 (USB_D+)
- net BT.D+: now also J5.2 (Pin_2)
- net BT.D-: now reaches U4.18 (USB_D-)
- net BT.D-: now also J5.3 (Pin_3)
- new net +5V: J5.1 (Pin_1)
- new net LCD.DC: U8.5 (DC/RS)
- new net LCD.LED: U8.8 (LED)
- new net LCD.~{RST}: U8.4 (~{RESET})
- no-connect marks 8 -> 6
Other:
- note added: "Schematic Labels"
- moved on the sheet: J1, J6

Commit message: Revert "PCB update - Minh"
This reverts commit 0608947e49f54a64abc006b190e3b029bac40ad1.
Parts:
- removed J5: BT USB Debug, symbol Connector:Conn_01x04_Pin
- removed J7: UART Debug, symbol Connector:Conn_01x06_Pin
- removed U8: 362 TFT LCD, symbol ECE477_PartsLibrary:362_OLED
- added DS1: OLED-128O064D, Display:OLED-128O064D, symbol Display_Graphic:OLED-128O064D
Connections:
- net SPI.MISO: no longer J6.3 (Pin_3)
- net SPI.MOSI: no longer J6.2 (Pin_2)
- net SPI.SCLK: no longer J6.1 (Pin_1)
- net SPI.~{CS}: no longer J6.4 (Pin_4)
- net BT.D+: no longer names the net of U4.17 (USB_D+)
- net BT.D-: no longer names the net of U4.18 (USB_D-)
- new net: DS1.1 (GND), DS1.30 (GND)
- new net BT.MISO: J6.3 (Pin_3)
- new net BT.MOSI: J6.2 (Pin_2)
- new net BT.SCLK: J6.1 (Pin_1)
- new net BT.~{CS}: J6.4 (Pin_4)
- no-connect marks 6 -> 8
Other:
- note removed: "Schematic Labels"
- moved on the sheet: J1, J6
