File: PCB/peri.kicad_sch (KiCad schematic)
At the start: 6 parts, among them J1 Micro_SD_Card, J5 BT USB Debug, J6 SPI Debug, J7 UART Debug, U4 RN42, U8 362 TFT LCD

Commit message: PCB Update - Minh
Parts:
- added C15, C16, C17, C18, C19: 0.1u, symbol Device:C
- added D14, D15: BT LED, symbol Device:LED
- added J8: BT Mode Conn, symbol Connector_Generic:Conn_02x04_Counter_Clockwise
- added J9: BT IO Debug, symbol Connector:Conn_01x05_Pin
- added R27, R28: 470, symbol Device:R
- added R29, R30: 3k3, symbol Device:R
- added R32, R33: 300k, symbol Device:R
- added R34, R35: 100k, symbol Device:R
- added RN2: 3k3, symbol Device:R_Pack04
- added SW1, SW4: RST_PB, symbol Switch:SW_Push
Connections:
- net +3V3: now also C15.1, C16.1, C17.1, R27.2, R28.2, R29.1, R30.1, R32.1, R33.1, RN2.5 (R4.2), RN2.6 (R3.2), RN2.7 (R2.2), RN2.8 (R1.2)
- net BT.~{RST}: now also C19.2, R29.2, SW4.1
- net GND: now also C15.2, C16.2, C17.2, C18.1, C19.1, R34.2, R35.2, SW1.2, SW4.2
- net LCD.~{RST}: now also C18.2, R30.2, SW1.1
- net BT.GPIO2: now reaches U4.19 (GPIO2)
- net BT.GPIO2: now also J9.3 (Pin_3)
- net BT.GPIO3: now reaches U4.20 (GPIO3)
- net BT.GPIO3: now also J8.5 (Pin_5)
- net BT.GPIO5: now reaches U4.21 (GPIO5)
- net BT.GPIO5: now also D14.1 (K)
- net BT.GPIO4: now reaches U4.22 (GPIO4)
- net BT.GPIO4: now also J8.6 (Pin_6)
- net BT.GPIO6: now reaches U4.3 (GPIO6)
- net BT.GPIO6: now also J8.7 (Pin_7)
- net BT.AIO0: now reaches U4.30 (AIO0)
- net BT.AIO0: now also J9.5 (Pin_5), R33.2, R34.1
- net BT.GPIO8: now reaches U4.31 (GPIO8)
- net BT.GPIO8: now also D15.1 (K)
- net BT.GPIO9: now reaches U4.32 (GPIO9)
- net BT.GPIO9: now also J9.2 (Pin_2)
- net BT.GPIO10: now reaches U4.33 (GPIO10)
- net BT.GPIO10: now also J9.1 (Pin_1)
- net BT.AIO1: now reaches U4.35 (AIO1)
- net BT.AIO1: now also J9.4 (Pin_4), R32.2, R35.1
- net BT.GPIO7: now reaches U4.4 (GPIO7)
- net BT.GPIO7: now also J8.8 (Pin_8)
- new net: J8.1 (Pin_1), RN2.4 (R4.1)
- new net: J8.2 (Pin_2), RN2.3 (R3.1)
- new net: J8.3 (Pin_3), RN2.2 (R2.1)
- new net: J8.4 (Pin_4), RN2.1 (R1.1)
- new net: D14.2 (A), R27.1
- new net: D15.2 (A), R28.1
- no-connect marks 6 -> 7
Other:
- note added: "Bluetooth RN42"
- note added: "ECE362 TFT LCD"
- note added: "MicroSD Adapter"
- moved on the sheet: J1, J5, J6, J7, U4

Commit message: update
Parts:
- removed J1: Micro_SD_Card, symbol Connector:Micro_SD_Card
- removed J7: UART Debug, symbol Connector:Conn_01x06_Pin
- removed SW1, SW4: RST_PB, symbol Switch:SW_Push
- added J403: MEM2080-00-128-00-A_REVA, MEM2080-00-128-00-A_REVA:GCT_MEM2080-00-128-00-A_REVA, symbol ECE477_PartsLibrary:MEM2080-00-128-00-A_REVA
- added J406: Conn_01x03_Pin, Connector_PinHeader_2.54mm:PinHeader_1x03_P2.54mm_Vertical, symbol Connector:Conn_01x03_Pin
- added J407, J408: Conn_01x04_Pin, Connector_PinHeader_2.54mm:PinHeader_1x04_P2.54mm_Vertical, symbol Connector:Conn_01x04_Pin
- added R409: 0, Resistor_SMD:R_0603_1608Metric_Pad0.98x0.95mm_HandSolder, symbol Device:R
- added SW401, SW402: PTS647SM70SMTR2LFS, PTS647SM70SMTR2LFS_CNK, symbol ECE477_PartsLibrary:PTS647SM70SMTR2LFS
- C401: renamed from C19; footprint (none) -> Capacitor_SMD:C_0603_1608Metric_Pad1.08x0.95mm_HandSolder; DigiKey Part (none) -> 490-5405-1-ND
- C402: renamed from C15; footprint (none) -> Capacitor_SMD:C_0603_1608Metric_Pad1.08x0.95mm_HandSolder; DigiKey Part (none) -> 490-5405-1-ND
- C403: renamed from C16; footprint (none) -> Capacitor_SMD:C_0603_1608Metric_Pad1.08x0.95mm_HandSolder; DigiKey Part (none) -> 490-5405-1-ND
- C404: renamed from C17; footprint (none) -> Capacitor_SMD:C_0603_1608Metric_Pad1.08x0.95mm_HandSolder; DigiKey Part (none) -> 490-5405-1-ND
- C405: renamed from C18; footprint (none) -> Capacitor_SMD:C_0603_1608Metric_Pad1.08x0.95mm_HandSolder; DigiKey Part (none) -> 490-5405-1-ND
- D401: renamed from D14; footprint (none) -> LED_SMD:LED_0805_2012Metric_Pad1.15x1.40mm_HandSolder; DigiKey Part (none) -> 475-LSR976-NR-1CT-ND
- D402: renamed from D15; footprint (none) -> LED_SMD:LED_0805_2012Metric_Pad1.15x1.40mm_HandSolder; DigiKey Part (none) -> 475-LSR976-NR-1CT-ND
- J401: renamed from J9; footprint (none) -> Connector_PinHeader_2.54mm:PinHeader_1x05_P2.54mm_Vertical
- J402: renamed from J5; footprint (none) -> Connector_PinHeader_2.54mm:PinHeader_1x04_P2.54mm_Vertical
- J404: renamed from J6; footprint (none) -> Connector_PinHeader_2.54mm:PinHeader_1x06_P2.54mm_Vertical
- J405: renamed from J8; footprint (none) -> Connector_PinHeader_2.54mm:PinHeader_2x04_P2.54mm_Vertical
- R401: renamed from R27; footprint (none) -> Resistor_SMD:R_0603_1608Metric_Pad0.98x0.95mm_HandSolder; DigiKey Part (none) -> 13-RC0603FR-13470RLCT-ND
- R402: renamed from R28; footprint (none) -> Resistor_SMD:R_0603_1608Metric_Pad0.98x0.95mm_HandSolder; DigiKey Part (none) -> 13-RC0603FR-13470RLCT-ND
- R403: renamed from R29; footprint (none) -> Resistor_SMD:R_0603_1608Metric_Pad0.98x0.95mm_HandSolder; DigiKey Part (none) -> 13-RC0603FR-133K3LCT-ND
- R404: renamed from R32; footprint (none) -> Resistor_SMD:R_0603_1608Metric_Pad0.98x0.95mm_HandSolder; DigiKey Part (none) -> YAG2585CT-ND
- R405: renamed from R35; footprint (none) -> Resistor_SMD:R_0603_1608Metric_Pad0.98x0.95mm_HandSolder; DigiKey Part (none) -> 311-100KHRCT-ND
- R406: renamed from R33; footprint (none) -> Resistor_SMD:R_0603_1608Metric_Pad0.98x0.95mm_HandSolder; DigiKey Part (none) -> YAG2585CT-ND
- R407: renamed from R34; footprint (none) -> Resistor_SMD:R_0603_1608Metric_Pad0.98x0.95mm_HandSolder; DigiKey Part (none) -> 311-100KHRCT-ND
- R408: renamed from R30; footprint (none) -> Resistor_SMD:R_0603_1608Metric_Pad0.98x0.95mm_HandSolder; DigiKey Part (none) -> 13-RC0603FR-133K3LCT-ND
- RN401: renamed from RN2; footprint (none) -> Resistor_SMD:R_Array_Convex_4x1206; DigiKey Part (none) -> 13-YC164-FR-073K32LCT-ND
- U401: renamed from U4; value RN42 -> RN42HID-I/RM; DigiKey Part (none) -> RN42HID-I/RM-ND
- U402: renamed from U8; footprint (none) -> Connector_PinHeader_2.54mm:PinHeader_1x09_P2.54mm_Vertical
Connections:
- net +3V3: now also J403.P4 (VDD), J408.3 (Pin_3), R409.1
- net BT.RX: now also J408.2 (Pin_2)
- net BT.TX: now also J408.1 (Pin_1)
- net BT.~{RST}: now also SW401.1, SW401.2
- net GND: now also J403.DSW1 (LEVER_PIN), J403.P6 (VSS), J403.S1 (SHIELD), J403.S2 (SHIELD__1), J403.S3 (SHIELD__2), J403.S4 (SHIELD__3), J408.4 (Pin_4), SW401.3, SW401.4, SW402.3, SW402.4
- net LCD.~{RST}: now also SW402.1, SW402.2
- net BT.CTS: no longer names the net of U401.16 (UART_CTS)
- net BT.RTS: no longer names the net of U401.15 (UART_RTS)
- net LCD.LED: no longer names the net of U402.8 (LED)
- net LCD.LED: now also R409.2
- net SPI.MISO renamed BT.MISO
- net BT.MISO: no longer U402.6 (SDO/MISO)
- net SPI.MOSI renamed BT.MOSI
- net BT.MOSI: no longer U402.9 (SDI/MOSI)
- net SPI.SCLK renamed BT.SCLK
- net BT.SCLK: no longer U402.7 (SCK)
- net SPI.~{CS} renamed BT.~{CS}
- net BT.~{CS}: no longer U402.3 (CS)
- new net LCD.MOSI: J406.2 (Pin_2), U402.9 (SDI/MOSI)
- new net LCD.SCLK: J406.1 (Pin_1), U402.7 (SCK)
- new net LCD.~{CS}: J406.3 (Pin_3), U402.3 (CS)
- new net SD.CD: J403.DSW2 (SWITCH_PIN)
- new net SD.MISO: J403.P7 (DAT0), J407.3 (Pin_3)
- new net SD.MOSI: J403.P3 (CMD), J407.2 (Pin_2)
- new net SD.SCLK: J403.P5 (CLK), J407.1 (Pin_1)
- new net SD.~{CS}: J403.P2 (CD/DAT3), J407.4 (Pin_4)
- no-connect marks 7 -> 10

Commit message: Update 90% done
Parts:
- removed J401: BT IO Debug, Connector_PinHeader_2.54mm:PinHeader_1x05_P2.54mm_Vertical, symbol Connector:Conn_01x05_Pin
- removed J402: BT USB Debug, Connector_PinHeader_2.54mm:PinHeader_1x04_P2.54mm_Vertical, symbol Connector:Conn_01x04_Pin
- removed J404: SPI Debug, Connector_PinHeader_2.54mm:PinHeader_1x06_P2.54mm_Vertical, symbol Connector:Conn_01x06_Pin
- removed J408: Conn_01x04_Pin, Connector_PinHeader_2.54mm:PinHeader_1x04_P2.54mm_Vertical, symbol Connector:Conn_01x04_Pin
- added J401: Conn_02x05_Counter_Clockwise, Connector_PinHeader_2.54mm:PinHeader_2x05_P2.54mm_Vertical, symbol Connector_Generic:Conn_02x05_Counter_Clockwise
- added R410, R411: 3k3, Resistor_SMD:R_0603_1608Metric_Pad0.98x0.95mm_HandSolder, symbol Device:R
- added R412: 100k, Resistor_SMD:R_0603_1608Metric_Pad0.98x0.95mm_HandSolder, symbol Device:R
- C401, C402, C403, C404, C405: Manufacturer (none) -> Murata Electronics; Mfg. Part # (none) -> GRM033R61A104ME15D; Package (none) -> 0603; Supplier (none) -> DigiKey; Supplier Part # (none) -> 490-5405-1-ND
- D401, D402: Manufacturer (none) -> ams-OSRAM USA INC.; Mfg. Part # (none) -> LS R976-NR-1; Package (none) -> 0805; Supplier (none) -> DigiKey; Supplier Part # (none) -> 475-LSR976-NR-1CT-ND
- J405, U402: Supplier (none) -> Amazon
- J406: renamed from J407; Supplier (none) -> Amazon
- J407: renamed from J403; value MEM2080-00-128-00-A_REVA -> 1040310811; footprint MEM2080-00-128-00-A_REVA:GCT_MEM2080-00-128-00-A_REVA -> ECE477_PartsLibrary:MOLEX_104031-0811; symbol ECE477_PartsLibrary:MEM2080-00-128-00-A_REVA -> ECE477_PartsLibrary:104031-0811; DigiKey Part 2073-MEM2080-00-128-00-ACT-ND -> WM6357CT-ND; Manufacturer (none) -> Molex; Mfg. Part # (none) -> 1040310811; Package (none) -> MOLEX_104031-0811; Supplier (none) -> DigiKey; Supplier Part # (none) -> WM6357CT-ND
- J408: renamed from J406; Supplier (none) -> Amazon
- R401, R402: Manufacturer (none) -> YAGEO; Mfg. Part # (none) -> RC0603FR-13470RL; Package (none) -> 0603; Supplier (none) -> DigiKey; Supplier Part # (none) -> 13-RC0603FR-13470RLCT-ND
- R403: Manufacturer (none) -> YAGEO; Mfg. Part # (none) -> RC0603FR-133K3L; Package (none) -> 0603; Supplier (none) -> DigiKey; Supplier Part # (none) -> 13-RC0603FR-133K3LCT-ND
- R404, R406: Manufacturer (none) -> YAGEO; Mfg. Part # (none) -> RC0603FR-07300KL; Package (none) -> 0603; Supplier (none) -> DigiKey; Supplier Part # (none) -> 311-300KHRCT-ND
- R405, R407: Manufacturer (none) -> YAGEO; Mfg. Part # (none) -> RC0603FR-07100KL; Package (none) -> 0603; Supplier (none) -> DigiKey; Supplier Part # (none) -> 311-100KHRCT-ND
- R408: renamed from R409; Manufacturer (none) -> YAGEO; Mfg. Part # (none) -> RC0603JR-070RL; Package (none) -> 0603; Supplier (none) -> DigiKey; Supplier Part # (none) -> 311-0.0GRCT-ND
- R409: renamed from R408; Manufacturer (none) -> YAGEO; Mfg. Part # (none) -> RC0603FR-133K3L; Package (none) -> 0603; Supplier (none) -> DigiKey; Supplier Part # (none) -> 13-RC0603FR-133K3LCT-ND
- RN401: Manufacturer (none) -> YAGEO; Mfg. Part # (none) -> YC164-FR-073K32L; Package (none) -> 4x1206_Convex; Supplier (none) -> DigiKey; Supplier Part # (none) -> 13-YC164-FR-073K32LCT-ND
- SW401, SW402: footprint PTS647SM70SMTR2LFS_CNK -> ECE477_PartsLibrary:PTS647SM70SMTR2LFS_CNK; Manufacturer (none) -> C&K; Mfg. Part # (none) -> PTS 647 SM70 SMTR2 LFS; Package (none) -> PTS647SM70SMTR2LFS_CNK; Supplier (none) -> DigiKey; Supplier Part # (none) -> PTS647SM70SMTR2LFSCT-ND
- U401: Manufacturer (none) -> Microchip Technology; Mfg. Part # (none) -> RN42HID-I/RM; Package (none) -> RN42; Supplier (none) -> DigiKey; Supplier Part # (none) -> RN42HID-I/RM-ND
Connections:
- net +3V3: now also J407.4 (VDD), J407.9 (SW-1), J401.10 (Pin_10); no longer J407.P4 (VDD)
- net BT.D+: now also J401.3 (Pin_3)
- net BT.D-: now also J401.4 (Pin_4)
- net BT.MISO: now also J401.7 (Pin_7)
- net BT.MOSI: now also J401.8 (Pin_8)
- net BT.RX: now also J401.2 (Pin_2), R410.2; no longer U401.13 (UART_RX)
- net BT.SCLK: now also J401.9 (Pin_9)
- net BT.TX: now also J401.1 (Pin_1), R411.2; no longer U401.14 (UART_TX)
- net BT.~{CS}: now also J401.6 (Pin_6)
- net GND: now also J407.6 (VSS), J407.G1 (GND__1), J407.G2 (GND__2), J407.G3 (GND__3), J407.G4 (GND__4), J401.5 (Pin_5), R412.1; no longer J407.DSW1 (LEVER_PIN), J407.P6 (VSS), J407.S1 (SHIELD), J407.S2 (SHIELD__1), J407.S3 (SHIELD__2), J407.S4 (SHIELD__3)
- net SD.CD: now also J407.10 (SW-2), R412.2; no longer J407.DSW2 (SWITCH_PIN)
- net SD.MISO: now also J406.1 (Pin_1), J407.7 (DAT0); no longer J406.3 (Pin_3), J407.P7 (DAT0)
- net SD.MOSI: now also J406.3 (Pin_3), J407.3 (CMD); no longer J406.2 (Pin_2), J407.P3 (CMD)
- net SD.SCLK: now also J406.2 (Pin_2), J407.5 (CLK); no longer J406.1 (Pin_1), J407.P5 (CLK)
- net SD.~{CS}: now also J407.2 (CD/DAT3); no longer J407.P2 (CD/DAT3)
- new net: R410.1, U401.13 (UART_RX)
- new net: R411.1, U401.14 (UART_TX)

Commit message: design 02/17
Parts:
- removed C405: 0.1u, Capacitor_SMD:C_0603_1608Metric_Pad1.08x0.95mm_HandSolder, symbol Device:C
- removed J405: BT Mode Conn, Connector_PinHeader_2.54mm:PinHeader_2x04_P2.54mm_Vertical, symbol Connector_Generic:Conn_02x04_Counter_Clockwise
- removed SW402: PTS647SM70SMTR2LFS, ECE477_PartsLibrary:PTS647SM70SMTR2LFS_CNK, symbol ECE477_PartsLibrary:PTS647SM70SMTR2LFS
- added J405: BT Mode Conn, Connector_PinHeader_2.54mm:PinHeader_2x04_P2.54mm_Vertical, symbol Connector_Generic:Conn_02x04_Odd_Even
- J401: footprint Connector_PinHeader_2.54mm:PinHeader_2x05_P2.54mm_Vertical -> Connector_PinHeader_2.54mm:PinHeader_2x06_P2.54mm_Vertical; symbol Connector_Generic:Conn_02x05_Counter_Clockwise -> Connector_Generic:Conn_02x06_Odd_Even; Supplier (none) -> Amazon
Connections:
- net +3V3: now also J401.1 (Pin_1); no longer J401.10 (Pin_10)
- net BT.D+: now also J401.5 (Pin_5); no longer J401.3 (Pin_3)
- net BT.D-: now also J401.3 (Pin_3); no longer J401.4 (Pin_4)
- net BT.GPIO3: now also J405.1 (Pin_1)
- net BT.GPIO4: now also J405.3 (Pin_3)
- net BT.GPIO6: now also J405.5 (Pin_5)
- net BT.GPIO7: now also J405.7 (Pin_7)
- net BT.MISO: now also J401.6 (Pin_6); no longer J401.7 (Pin_7)
- net BT.MOSI: now also J401.4 (Pin_4); no longer J401.8 (Pin_8)
- net BT.RX: now also J401.9 (Pin_9); no longer J401.2 (Pin_2), R410.2
- net BT.SCLK: now also J401.2 (Pin_2); no longer J401.9 (Pin_9)
- net BT.TX: now also J401.11 (Pin_11); no longer J401.1 (Pin_1), R411.2
- net BT.~{CS}: now also J401.8 (Pin_8); no longer J401.6 (Pin_6)
- net GND: now also J401.7 (Pin_7); no longer J401.5 (Pin_5)
- net LCD.MOSI: now also J408.1 (Pin_1); no longer J408.2 (Pin_2)
- net LCD.SCLK: now also J408.2 (Pin_2); no longer J408.1 (Pin_1)
- net at RN401.4 (R4.1): now also J405.2 (Pin_2)
- net at RN401.3 (R3.1): now also J405.4 (Pin_4)
- net at RN401.2 (R2.1): now also J405.6 (Pin_6)
- net at RN401.1 (R1.1): now also J405.8 (Pin_8)
- net BT.GPIO10: no longer names the net of U401.33 (GPIO10)
- net BT.GPIO2: no longer names the net of U401.19 (GPIO2)
- net BT.GPIO9: no longer names the net of U401.32 (GPIO9)
- new net CONN.RX: J401.12 (Pin_12), R410.2
- new net CONN.TX: J401.10 (Pin_10), R411.2
- no-connect marks 10 -> 13

Commit message: Update Rev 2
Parts:
- removed R408: 0, Resistor_SMD:R_0603_1608Metric_Pad0.98x0.95mm_HandSolder, symbol Device:R
Connections:
- net +3V3: now also U402.8 (LED)
Other:
- company: (none) -> ECE477 - Team 4: KayO
- title: (none) -> Peripherals
Changed lines of the file:
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@@
 (kicad_sch (version 20230121) (generator eeschema)
-  (paper "A4")
+  (paper "A3")
+  (title_block
+    (title "Peripherals")
+    (date "2024-02-21")
+    (rev "2")
+    (company "ECE477 - Team 4: KayO")
+  )
   (junction (at 63.5 170.18) (diameter 0) (color 0 0 0 0)
   )
@@
     (stroke (width 0) (type default))
   )
-  (bus (pts (xy 222.25 132.08) (xy 231.14 132.08))
+  (bus (pts (xy 345.44 219.075) (xy 354.33 219.075))
     (stroke (width 0) (type default))
   )
@@
     (stroke (width 0) (type default))
   )
-  (wire (pts (xy 220.98 64.77) (xy 233.68 64.77))
-    (stroke (width 0) (type default))
-  )
   (wire (pts (xy 45.72 106.68) (xy 49.53 106.68))
     (stroke (width 0) (type default))
@@
     (stroke (width 0) (type default))
   )
-  (bus (pts (xy 222.25 137.16) (xy 231.14 137.16))
+  (bus (pts (xy 345.44 224.155) (xy 354.33 224.155))
     (stroke (width 0) (type default))
   )
@@
     (stroke (width 0) (type default))
   )
-  (bus (pts (xy 222.25 142.24) (xy 231.14 142.24))
-    (stroke (width 0) (type default))
-  )
-  (wire (pts (xy 212.09 64.77) (xy 213.36 64.77))
+  (bus (pts (xy 345.44 229.235) (xy 354.33 229.235))
+    (stroke (width 0) (type default))
+  )
+  (wire (pts (xy 212.09 64.77) (xy 233.68 64.77))
     (stroke (width 0) (type default))
   )
@@
     (fill (type none))
   )
-  (rectangle (start 167.64 128.27) (end 281.94 162.56)
+  (rectangle (start 290.83 215.265) (end 405.13 249.555)
     (stroke (width 0) (type default))
     (fill (type none))
@@
     (effects (font (face "KiCad Font") (size 1.27 1.27) (thickness 0.254) bold) (justify left bottom))
   )
-  (text "Schematic Labels" (at 168.91 127 0)
+  (text "Schematic Labels" (at 292.1 213.995 0)
     (effects (font (face "KiCad Font") (size 1.27 1.27) (thickness 0.254) bold) (justify left bottom))
   )
@@
     )
   )
-  (global_label "BT{TX, RX, ~{RST}, GPIO[3..4], GPIO[6..7]}" (shape bidirectional) (at 222.25 132.08 180) (fields_autoplaced)
-    (effects (font (size 1.27 1.27)) (justify right))
-    (property "Intersheetrefs" "${INTERSHEET_REFS}" (at 180.2346 132.08 0)
+  (global_label "BT{TX, RX, ~{RST}, GPIO[3..4], GPIO[6..7]}" (shape bidirectional) (at 345.44 219.075 180) (fields_autoplaced)
+    (effects (font (size 1.27 1.27)) (justify right))
+    (property "Intersheetrefs" "${INTERSHEET_REFS}" (at 303.4246 219.075 0)
       (effects (font (size 1.27 1.27)) (justify right) hide)
     )
@@
     )
   )
-  (global_label "SD{SCLK, MOSI, MISO, ~{CS}, CD}" (shape bidirectional) (at 222.25 137.16 180) (fields_autoplaced)
-    (effects (font (size 1.27 1.27)) (justify right))
-    (property "Intersheetrefs" "${INTERSHEET_REFS}" (at 188.7015 137.16 0)
+  (global_label "SD{SCLK, MOSI, MISO, ~{CS}, CD}" (shape bidirectional) (at 345.44 224.155 180) (fields_autoplaced)
+    (effects (font (size 1.27 1.27)) (justify right))
+    (property "Intersheetrefs" "${INTERSHEET_REFS}" (at 311.8915 224.155 0)
       (effects (font (size 1.27 1.27)) (justify right) hide)
     )
@@
     )
   )
-  (global_label "LCD{SCLK, MOSI, ~{CS}, DC, ~{RST}}" (shape bidirectional) (at 222.25 142.24 180) (fields_autoplaced)
-    (effects (font (size 1.27 1.27)) (justify right))
-    (property "Intersheetrefs" "${INTERSHEET_REFS}" (at 188.762 142.24 0)
+  (global_label "LCD{SCLK, MOSI, ~{CS}, DC, ~{RST}}" (shape bidirectional) (at 345.44 229.235 180) (fields_autoplaced)
+    (effects (font (size 1.27 1.27)) (justify right))
+    (property "Intersheetrefs" "${INTERSHEET_REFS}" (at 311.952 229.235 0)
       (effects (font (size 1.27 1.27)) (justify right) hide)
     )
@@
     )
   )
-  (hierarchical_label "LCD{SCLK, MOSI, ~{CS}, DC, ~{RST}}" (shape bidirectional) (at 231.14 142.24 0) (fields_autoplaced)
-    (effects (font (size 1.27 1.27)) (justify left))
-  )
-  (hierarchical_label "BT{TX, RX, ~{RST}, GPIO[3..4], GPIO[6..7]}" (shape bidirectional) (at 231.14 132.08 0) (fields_autoplaced)
-    (effects (font (size 1.27 1.27)) (justify left))
-  )
-  (hierarchical_label "SD{SCLK, MOSI, MISO, ~{CS}, CD}" (shape bidirectional) (at 231.14 137.16 0) (fields_autoplaced)
+  (hierarchical_label "LCD{SCLK, MOSI, ~{CS}, DC, ~{RST}}" (shape bidirectional) (at 354.33 229.235 0) (fields_autoplaced)
+    (effects (font (size 1.27 1.27)) (justify left))
+  )
+  (hierarchical_label "BT{TX, RX, ~{RST}, GPIO[3..4], GPIO[6..7]}" (shape bidirectional) (at 354.33 219.075 0) (fields_autoplaced)
+    (effects (font (size 1.27 1.27)) (justify left))
+  )
+  (hierarchical_label "SD{SCLK, MOSI, MISO, ~{CS}, CD}" (shape bidirectional) (at 354.33 224.155 0) (fields_autoplaced)
     (effects (font (size 1.27 1.27)) (justify left))
   )
@@
         )
       )
-    )
-  )
-  (symbol (lib_id "Device:R") (at 217.17 64.77 90) (unit 1)
-    (in_bom yes) (on_board yes) (dnp no)
-    (property "Reference" "R408" (at 217.17 62.23 90)
-      (effects (font (size 1.27 1.27)))
-    )
-    (property "Value" "0" (at 217.17 64.77 90)
-      (effects (font (size 1.27 1.27)))
-    )
-    (property "Footprint" "Resistor_SMD:R_0603_1608Metric_Pad0.98x0.95mm_HandSolder" (at 217.17 66.548 90)
-      (effects (font (size 1.27 1.27)) hide)
-    )
-    (property "Datasheet" "~" (at 217.17 64.77 0)
-      (effects (font (size 1.27 1.27)) hide)
-    )
-    (property "DigiKey Part" "311-0.0GRCT-ND" (at 217.17 64.77 0)
-      (effects (font (size 1.27 1.27)) hide)
-    )
-    (property "Description" "RES 0 OHM JUMPER 1/10W 0603" (at 217.17 64.77 0)
-      (effects (font (size 1.27 1.27)) hide)
-    )
-    (property "Manufacturer" "YAGEO" (at 217.17 64.77 0)
-      (effects (font (size 1.27 1.27)) hide)
-    )
-    (property "Mfg. Part #" "RC0603JR-070RL" (at 217.17 64.77 0)
-      (effects (font (size 1.27 1.27)) hide)
-    )
-    (property "Supplier" "DigiKey" (at 217.17 64.77 0)
-      (effects (font (size 1.27 1.27)) hide)
-    )
-    (property "Supplier Part #" "311-0.0GRCT-ND" (at 217.17 64.77 0)
-      (effects (font (size 1.27 1.27)) hide)
-    )
-    (property "Package" "0603" (at 217.17 64.77 0)
-      (effects (font (size 1.27 1.27)) hide)
-    )
-    (pin "1")
-    (pin "2")
-    (instances
-      (project "ECE477_PCBDesign"
-        (path "/a3f06f97-9851-42dd-ac9b-8261120cb59a/4cedef9a-026c-4a65-adba-5aed83578928"
-          (reference "R408") (unit 1)
-        )
-      )
