File: PCB/peri.kicad_sch (KiCad schematic)
At the start: 26 parts, among them J401 Conn_02x05_Counter_Clockwise, J402 Conn_01x06_Pin, J406 Conn_01x04_Pin, J407 1040310811, J408 Conn_01x03_Pin, Q401 SS8050-G, Q402 SS8050-G, SW401 PTS647SM70SMTR2LFS, SW402 PTS647SM70SMTR2LFS, U402 362 TFT LCD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

Commit message: PCB Update
Parts:
- added D401, D402, D403, D404, D407, D408, D409, D410, D411, D412: D5V0L1B2WS-7, Diode_SMD:D_SOD-323_HandSoldering, symbol Device:D_TVS
- added SW403, SW404: SW_Push, Connector_JST:JST_XH_B2B-XH-A_1x02_P2.50mm_Vertical, symbol Switch:SW_SPST
Connections:
- net +3V3: now also SW404.2 (B)
- net BT.EN: now also SW403.1 (A)
- net GND: now also D401.1 (A1), D402.1 (A1), D403.1 (A1), D404.1 (A1), D407.1 (A1), D408.1 (A1), D409.1 (A1), D410.1 (A1), D411.1 (A1), D412.1 (A1), SW403.2 (B)
- net LCD.DC: now also D409.2 (A2)
- net LCD.MOSI: now also D411.2 (A2)
- net LCD.SCLK: now also D412.2 (A2)
- net LCD.~{CS}: now also D410.2 (A2)
- net LCD.~{RST}: now also D408.2 (A2)
- net SD.CD: now also D401.2 (A2)
- net SD.MISO: now also D403.2 (A2)
- net SD.MOSI: now also D404.2 (A2)
- net SD.SCLK: now also D407.2 (A2)
- net SD.~{CS}: now also D402.2 (A2)
- net at D405.2 (A), U403.36 (IO22): now also SW404.1 (A)
Other:
- moved on the sheet: C403, D406, J406, J407, R412, R416
