File: PCB/ECE477_PCBDesign.kicad_pcb (KiCad board)
At the start: 2 copper layers, 172 parts, among them J202 Conn_01x02_Pin, J203 Conn_01x02_Pin, J204 USB_C_Receptacle_USB2.0_16P, J301 USB_C_Receptacle_USB2.0_16P, J302 Conn_01x05_Pin, J304 Conn_01x07_Pin, J401 BT IO Debug, J402 BT USB Debug, J404 SPI Debug, J405 BT Mode Conn, J406 Conn_01x03_Pin, J407 Conn_01x04_Pin, J408 Conn_01x04_Pin, Q201 MMBT2222A, Q202 MMBT2222A, Q203 MMBT2222A, Q204 MMBT2222A, Q205 MMBT2222A, SW201 SW_SPST, SW203 SW_SPST, SW501 SW_Push, SW502 SW_Push, SW503 SW_Push, SW504 SW_Push, SW505 SW_Push, SW506 SW_Push, SW507 SW_Push, SW508 SW_Push, SW509 SW_Push, SW510 SW_Push, SW511 SW_Push, SW512 SW_Push, SW513 SW_Push, SW514 SW_Push, SW515 SW_Push, SW516 SW_Push, SW517 SW_Push, SW518 SW_Push, U202 TPS63031DSK, U203 BQ27441DRZR-G1A, U205 BQ24075RGT, U301 STM32F411RETx, U302 STM32F103CBTx, U401 RN42, U402 362 TFT LCD

Commit message: Update 90% done
Parts:
- removed BT201: Battery_Cell, Connector_JST:JST_PH_S2B-PH-SM4-TB_1x02-1MP_P2.00mm_Horizontal
- removed C212: 0.1u, Capacitor_SMD:C_0603_1608Metric_Pad1.08x0.95mm_HandSolder
- removed D211: SYSPWR_LED, LED_SMD:LED_0805_2012Metric_Pad1.15x1.40mm_HandSolder
- removed D303: D5V0L1B2S9-7, Diode_SMD:D_SOD-923
- removed J301: USB_C_Receptacle_USB2.0_16P, Connector_USB:USB_C_Receptacle_HRO_TYPE-C-31-M-12
- removed J304: Conn_01x07_Pin, Connector_PinHeader_2.54mm:PinHeader_1x07_P2.54mm_Vertical
- removed J402: BT USB Debug, Connector_PinHeader_2.54mm:PinHeader_1x04_P2.54mm_Vertical
- removed J404: SPI Debug, Connector_PinHeader_2.54mm:PinHeader_1x06_P2.54mm_Vertical
- removed R314, R316: 180, Resistor_SMD:R_0603_1608Metric_Pad0.98x0.95mm_HandSolder
- removed SW203: SW_SPST, Connector_JST:JST_XH_B2B-XH-A_1x02_P2.50mm_Vertical
- added C316: 0.1u, Capacitor_SMD:C_0603_1608Metric_Pad1.08x0.95mm_HandSolder, B.Cu at (173.4, 70.3)
- added C317: 0.1u, Capacitor_SMD:C_0603_1608Metric_Pad1.08x0.95mm_HandSolder, F.Cu at (169.1, 78.2)
- added C318: 0.1u, Capacitor_SMD:C_0603_1608Metric_Pad1.08x0.95mm_HandSolder, F.Cu at (178.1, 81.8)
- added C319: 0.1u, Capacitor_SMD:C_0603_1608Metric_Pad1.08x0.95mm_HandSolder, B.Cu at (179.2, 76.5)
- added C320: 0.1u, Capacitor_SMD:C_0603_1608Metric_Pad1.08x0.95mm_HandSolder, B.Cu at (179.2, 72.5)
- added D207: CHG_LED, LED_SMD:LED_0805_2012Metric_Pad1.15x1.40mm_HandSolder, F.Cu at (126.0, 63.6)
- added D208: PGOOD_LED, LED_SMD:LED_0805_2012Metric_Pad1.15x1.40mm_HandSolder, F.Cu at (132.3, 63.6)
- added J201: USB_C_Receptacle_USB2.0_16P, Connector_USB:USB_C_Receptacle_HRO_TYPE-C-31-M-12, F.Cu at (150.7, 62.5)
- added J206: Conn_01x10_Socket, ECE477_PartsLibrary:ECE477_BATBabySitter, F.Cu at (113.0, 79.7)
- added J303: STLink Connector, ECE477_PartsLibrary:CONN10_302-S101_OST, F.Cu at (208.3, 77.6)
- added JP201: Jumper_2_Open, Jumper:SolderJumper-2_P1.3mm_Open_Pad1.0x1.5mm, F.Cu at (112.4, 100.8)
- added JP202: Jumper_2_Bridged, Jumper:SolderJumper-2_P1.3mm_Bridged_Pad1.0x1.5mm, F.Cu at (121.9, 98.6)
- added JP203: Jumper_2_Open, Jumper:SolderJumper-2_P1.3mm_Open_Pad1.0x1.5mm, F.Cu at (103.4, 105.2)
- added JP204: Jumper_2_Bridged, Jumper:SolderJumper-2_P1.3mm_Bridged_Pad1.0x1.5mm, F.Cu at (136.6, 99.2)
- added L201: 1u, ECE477_PartsLibrary:IND_XFL4020-102MEC, F.Cu at (111.7, 105.1)
- added L202: 0.47u, ECE477_PartsLibrary:IND_IHLP-2020CZ, F.Cu at (128.6, 94.9)
- added R227: 590, Resistor_SMD:R_0603_1608Metric_Pad0.98x0.95mm_HandSolder, B.Cu at (131.6, 75.8)
- added R228: 1.5k, Resistor_SMD:R_0603_1608Metric_Pad0.98x0.95mm_HandSolder, B.Cu at (128.2, 80.9)
- added R229: 22, Resistor_SMD:R_0603_1608Metric_Pad0.98x0.95mm_HandSolder, B.Cu at (132.3, 73.5)
- added R410: 3k3, Resistor_SMD:R_0603_1608Metric_Pad0.98x0.95mm_HandSolder, F.Cu at (198.6, 101.0)
- added R411: 3k3, Resistor_SMD:R_0603_1608Metric_Pad0.98x0.95mm_HandSolder, F.Cu at (198.6, 103.0)
- added R412: 100k, Resistor_SMD:R_0603_1608Metric_Pad0.98x0.95mm_HandSolder, F.Cu at (102.7, 92.3)
- added SW202: SW_SPST, Connector_JST:JST_XH_B2B-XH-A_1x02_P2.50mm_Vertical, F.Cu at (95.8, 74.6)
- added SW301: PTS647SM70SMTR2LFS, ECE477_PartsLibrary:PTS647SM70SMTR2LFS_CNK, F.Cu at (181.0, 89.9)
- added SW302: PTS647SM70SMTR2LFS, ECE477_PartsLibrary:PTS647SM70SMTR2LFS_CNK, F.Cu at (184.2, 68.3)
- added SW303: SW_DPDT_x2, ECE477_PartsLibrary:SW_JS202011SCQN, F.Cu at (150.4, 79.4)
- added SW305: 1-1825010-3, ECE477_PartsLibrary:SW_1-1825010-3, F.Cu at (194.0, 71.4)
- added SW401: PTS647SM70SMTR2LFS, ECE477_PartsLibrary:PTS647SM70SMTR2LFS_CNK, F.Cu at (205.8, 104.5)
- added SW402: PTS647SM70SMTR2LFS, ECE477_PartsLibrary:PTS647SM70SMTR2LFS_CNK, F.Cu at (115.3, 120.9)
- added U201: LMS33460MG, ECE477_PartsLibrary:SOT65P210X110-5N, F.Cu at (119.7, 63.5)
- added U204: TPS63802DLAR, ECE477_PartsLibrary:VREG_TPS63802DLAR, F.Cu at (128.6, 100.0)
- added U303: LTST-C155KGJRKT, ECE477_PartsLibrary:SON4_LTST-C155KGJRKT_LTO, F.Cu at (172.6, 63.1)
- added X301: CG04874-8M, ECE477_PartsLibrary:XTAL_CG04874_NDK, F.Cu at (179.6, 95.2)
- added X302: CG04874-8M, ECE477_PartsLibrary:XTAL_CG04874_NDK, F.Cu at (182.8, 75.2)
- C201: value 10u -> 0.1u; moved to B.Cu
- C202, C207, C306, C307, C308, C309, C311, C312, C313, C314, C315, C401, C402, C403, C405, FB301, Q201, R203, R218, R219, R221, R301, R305, R403, R404, R405, R406, R407, RN201, RN401: moved to B.Cu
- C203: value 22u -> 10u
- C204: value 1u -> 22u
- C205: value 10u -> 1u
- C206, C209: value 10u -> 22u
- C210: value 1u -> 10u
- C211: value 0.1u -> 1u
- C301, C302: value 20p -> 0.1u; moved to B.Cu
- C303, C304: value 0.1u -> 20p; moved to B.Cu
- D201, D203, D301: value D5V0L1B2S9-7 -> D5V0L1B2T-7; footprint Diode_SMD:D_SOD-923 -> Diode_SMD:D_SOD-523; moved to B.Cu
- D204: value 3VDetect_LED -> D5V0L1B2T-7; footprint Diode_SMD:D_0805_2012Metric_Pad1.15x1.40mm_HandSolder -> Diode_SMD:D_SOD-523; moved to B.Cu
- D205: value PMEG4010BEA,115 -> 3VDetect_LED; footprint Diode_SMD:D_SOD-323 -> Diode_SMD:D_0805_2012Metric_Pad1.15x1.40mm_HandSolder
- D206, D302: value D5V0L1B2S9-7 -> 3757-SS12L_R1_00001CT-ND; footprint Diode_SMD:D_SOD-923 -> Diode_SMD:D_SMA; moved to B.Cu
- D209: value CHG_LED -> SYSPWR_LED
- D210: value PGOOD_LED -> 3757-SS12L_R1_00001CT-ND; footprint LED_SMD:LED_0805_2012Metric_Pad1.15x1.40mm_HandSolder -> Diode_SMD:D_SMA; moved to B.Cu
- D501, D502, D503, D504, D505, D506, D507, D508, D509, D510, D511, D512, D513, D514, D515, D516: value PMEG4010BEA,115 -> 3757-SS12L_R1_00001CT-ND; footprint Diode_SMD:D_SOD-323 -> Diode_SMD:D_SMA; moved to B.Cu
- J202: footprint Connector_PinHeader_2.54mm:PinHeader_1x02_P2.54mm_Vertical -> ECE477_PartsLibrary:CONN_S2B-PH-K-S_JST
- J204: value USB_C_Receptacle_USB2.0_16P -> Conn_01x02_Pin; footprint Connector_USB:USB_C_Receptacle_HRO_TYPE-C-31-M-12 -> Connector_PinHeader_2.54mm:PinHeader_1x02_P2.54mm_Vertical
- J302: value Conn_01x05_Pin -> Conn_01x03_Pin; footprint Connector_PinHeader_2.54mm:PinHeader_1x05_P2.54mm_Vertical -> Connector_PinHeader_2.54mm:PinHeader_1x03_P2.54mm_Vertical
- J401: value BT IO Debug -> Conn_02x05_Counter_Clockwise; footprint Connector_PinHeader_2.54mm:PinHeader_1x05_P2.54mm_Vertical -> Connector_PinHeader_2.54mm:PinHeader_2x05_P2.54mm_Vertical
- J406: value Conn_01x03_Pin -> Conn_01x04_Pin; footprint Connector_PinHeader_2.54mm:PinHeader_1x03_P2.54mm_Vertical -> Connector_PinHeader_2.54mm:PinHeader_1x04_P2.54mm_Vertical
- J407: value Conn_01x04_Pin -> 1040310811; footprint Connector_PinHeader_2.54mm:PinHeader_1x04_P2.54mm_Vertical -> ECE477_PartsLibrary:MOLEX_104031-0811
- J408: value Conn_01x04_Pin -> Conn_01x03_Pin; footprint Connector_PinHeader_2.54mm:PinHeader_1x04_P2.54mm_Vertical -> Connector_PinHeader_2.54mm:PinHeader_1x03_P2.54mm_Vertical
- R201: value 750 -> 100k; moved to B.Cu
- R202: value 5.1k -> 750
- R204: value 100k -> 5.1k; moved to B.Cu
- R209: value 1k -> 453k
- R210: value 10k -> 100k
- R211: value 511k -> 1k; moved to B.Cu
- R212: value 91k -> 10k; moved to B.Cu
- R213: value 10k -> 511k
- R214: value 10k -> 91k
- R215: value 1k -> 1M
- R216, R217: value 1k -> 10k; moved to B.Cu
- R220: value 180 -> 1k; moved to B.Cu
- R222: value 750 -> 1k; moved to B.Cu
- R223: value 10k -> 180
- R224: value 490 -> 1k
- R225: value 1.5k -> 750
- R226: value 22 -> 10k; moved to B.Cu
- R306: value 10k -> 4.7k
- R307: value 100k -> 2.7k
- R308: value 4.7k -> 10k; moved to B.Cu
- R309: value 4.7k -> 100k
- R310: value 2.7k -> 180
- R311: value 4.7k -> 180
- R312, R313: value 5.1k -> 4.7k; moved to B.Cu
- R408: value 3k3 -> 0
- R409: value 0 -> 3k3; moved to B.Cu
- U202: value TPS63031DSK -> TPS63021DSJR; footprint Package_SON:WSON-10-1EP_2.5x2.5mm_P0.5mm_EP1.2x2mm -> ECE477_PartsLibrary:IC_TPS63021DSJR
- U205: value BQ24075RGT -> BQ24075RGTR; footprint Package_DFN_QFN:VQFN-16-1EP_3x3mm_P0.5mm_EP1.6x1.6mm -> Package_DFN_QFN:VQFN-16-1EP_3x3mm_P0.5mm_EP1.6x1.6mm_ThermalVias
- U301: value STM32F411RETx -> STM32F411RET6
- U302: value STM32F103CBTx -> STM32F103CBT6
- U401: value RN42 -> RN42HID-I/RM
- moved SW517 161.5 mm to (202.2, 122.0)
- moved SW518 156.3 mm to (202.2, 113.0)
- moved SW516 156.1 mm to (193.2, 122.0)
- moved SW508 155.8 mm to (175.2, 122.0)
- moved SW515 155.6 mm to (193.2, 113.0)
- moved SW507 155.2 mm to (175.2, 113.0)
- moved SW512 150.8 mm to (184.2, 122.0)
- moved SW511 150.4 mm to (184.2, 113.0)
- moved SW504 148.8 mm to (166.2, 122.0)
- moved SW502 148.5 mm to (157.2, 122.0)
- moved SW503 148.3 mm to (166.2, 113.0)
- moved SW501 147.9 mm to (157.2, 113.0)
- moved C314 138.6 mm to (210.5, 68.3), turned to -90 degrees
- moved D516 136.9 mm to (195.2, 125.9), turned to 180 degrees
- moved R401 135.8 mm to (212.6, 106.5), turned to -90 degrees
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Connections:
- C201 pad 1: Net-(JP201-B) -> V_RAW
- C202 pad 1: Net-(U202-EN) -> +5V
- C203 pad 1: Net-(JP202-B) -> Net-(JP201-B)
- C204 pad 1: GND -> /Power Supply Unit/PWR_JP
- C204 pad 2: Net-(BT201-+) -> GND
- C205 pad 1: Net-(JP203-A) -> GND
- C205 pad 2: GND -> Net-(J202-Pin_1)
- C208 pad 1: Net-(JP204-A) -> Net-(JP203-A)
- C209 pad 1: V_BAT -> /Power Supply Unit/3V_JP
- C210 pad 1: +5V -> V_BAT
- C211 pad 1: V_RAW -> +5V
- C301 pad 1: GND -> +3V3
- C301 pad 2: Net-(C301-Pad2) -> GND
- C302 pad 1: GND -> +3V3
- C302 pad 2: Net-(C302-Pad2) -> GND
- C303 pad 2: STM.NRST -> Net-(C303-Pad2)
- C304 pad 1: +3V3 -> GND
- C304 pad 2: GND -> Net-(C304-Pad2)
- C306 pad 1: +3V3 -> GND
- C306 pad 2: GND -> STM.NRST
- D204 pad 2: Net-(D204-A) -> +5V
- D205 pad 1: Net-(D205-K) -> GND
- D205 pad 2: +5V -> Net-(D205-A)
- D206 pad 1: GND -> Net-(D206-K)
- D210 pad 2: SYS.PWR -> V_RAW
- D301 pad 2: STLink.D+ -> +5V
- D302 pad 1: GND -> Net-(D302-K)
- D302 pad 2: STLink.D- -> V_RAW_STLink
- FB201 pad 1: V_RAW -> Net-(D210-K)
- FB301 pad 1: V_RAW_STLink -> Net-(D302-K)
- J202 pad 1: SYS.PWR -> Net-(J202-Pin_1)
- J202 pad 2: BAT.EN1 -> GND
- J203 pad 2: BAT.EN2 -> BAT.EN1
- J302 pad 1: +3V3 -> STLink.TX
- J302 pad 2: STM.SWCLK -> STLink.RX
- J401 pad 1: BT.GPIO10 -> BT.TX
- J401 pad 2: BT.GPIO9 -> BT.RX
- J401 pad 3: BT.GPIO2 -> BT.D+
- J401 pad 4: BT.AIO1 -> BT.D-
- J401 pad 5: BT.AIO0 -> GND
- J406 pad 1: LCD.SCLK -> SD.MISO
- J406 pad 2: LCD.MOSI -> SD.SCLK
- J406 pad 3: LCD.~{CS} -> SD.MOSI
- J407 pad 1: SD.SCLK -> unconnected-(J407-DAT2-Pad1)
- J407 pad 2: SD.MOSI -> SD.~{CS}
- J407 pad 3: SD.MISO -> SD.MOSI
- J407 pad 4: SD.~{CS} -> +3V3
- J408 pad 1: BT.TX -> LCD.SCLK
- J408 pad 2: BT.RX -> LCD.MOSI
- J408 pad 3: +3V3 -> LCD.~{CS}
- Q201 pad 1: Net-(D205-K) -> Net-(D206-K)
- R201 pad 1: +5V -> GND
- R201 pad 2: Net-(D202-A) -> BAT.OFF
- R202 pad 1: Net-(J204-CC1) -> +5V
- R202 pad 2: GND -> Net-(D202-A)
- R203 pad 1: GND -> Net-(J201-CC1)
- R203 pad 2: Net-(J204-CC2) -> GND
- R204 pad 2: BAT.OFF -> Net-(J201-CC2)
- R206 pad 2: Net-(D204-A) -> Net-(D205-A)
- R207 pad 2: Net-(BT201-+) -> Net-(J202-Pin_1)
- R208 pad 1: Net-(JP202-B) -> /Power Supply Unit/PWR_JP
- R209 pad 1: USB.Detect -> Net-(JP203-A)
- R209 pad 2: GND -> Net-(U202-FB)
- R210 pad 1: Net-(U203-BIN) -> Net-(U202-FB)
- R211 pad 1: Net-(JP204-A) -> USB.Detect
- R211 pad 2: Net-(U204-FB) -> GND
- R212 pad 1: Net-(U204-FB) -> Net-(U203-BIN)
- R213 pad 1: +3V3 -> /Power Supply Unit/3V_JP
- R213 pad 2: BAT.GPOUT -> Net-(U204-FB)
- R214 pad 1: GND -> Net-(U204-FB)
- R214 pad 2: BAT.~{CE} -> GND
- R215 pad 1: ~{CE} -> Net-(JP203-A)
- R215 pad 2: GND -> Net-(U202-PG)
- R216 pad 1: EN1 -> +3V3
- R216 pad 2: GND -> BAT.GPOUT
- R217 pad 1: BAT.EN1 -> GND
- R217 pad 2: GND -> BAT.~{CE}
- R218 pad 1: EN2 -> ~{CE}
- R219 pad 1: BAT.EN2 -> EN1
- R220 pad 1: Net-(D209-K) -> BAT.EN1
- R220 pad 2: ~{CHG} -> GND
- R221 pad 1: Net-(D210-K) -> EN2
- R221 pad 2: ~{PGOOD} -> GND
- R222 pad 1: Net-(D211-K) -> BAT.EN2
- R223 pad 1: GND -> Net-(D207-K)
- R223 pad 2: TS -> ~{CHG}
- R224 pad 1: GND -> Net-(D208-K)
- R224 pad 2: ISET -> ~{PGOOD}
- R225 pad 1: GND -> Net-(D209-K)
- R225 pad 2: ILIM -> GND
- R226 pad 1: Net-(Q205-E) -> GND
- R226 pad 2: GND -> TS
- R302 pad 1: Net-(C301-Pad2) -> Net-(C303-Pad2)
- R303 pad 2: Net-(C302-Pad2) -> Net-(C304-Pad2)
- R305 pad 1: GND -> +3V3
- R305 pad 2: Net-(U302-BOOT0) -> STLink.NRST
- R306 pad 2: Net-(U302-PC13) -> Net-(U302-PB3)
- R307 pad 1: +3V3 -> Net-(U302-PB3)
- R307 pad 2: STLink.NRST -> +5V
- R308 pad 1: Net-(U302-PA0) -> GND
- R308 pad 2: +3V3 -> Net-(U302-PC13)
- R309 pad 2: Net-(U302-PA0) -> Net-(U302-BOOT0)
- R310 pad 1: Net-(U302-PB3) -> STLink.LED
- R310 pad 2: +5V -> Net-(R310-Pad2)
- R311 pad 1: GND -> STLink.LED
- R311 pad 2: Net-(U302-PB3) -> Net-(R311-Pad2)
- R312 pad 1: Net-(J301-CC1) -> Net-(U302-PA0)
- R312 pad 2: GND -> +3V3
- R313 pad 2: Net-(J301-CC2) -> Net-(U302-PA0)
- R408 pad 2: LCD.~{RST} -> Net-(U402-LED)
- R409 pad 2: Net-(U402-LED) -> LCD.~{RST}
- U202 pad 1: Net-(JP203-A) -> GND
- U202 pad 10: Net-(JP203-A) -> Net-(JP201-B)
- U202 pad 11: GND -> Net-(JP201-B)
- U202 pad 2: Net-(U202-L2) -> GND
- U202 pad 3: GND -> Net-(U202-FB)
- U202 pad 4: Net-(U202-L1) -> Net-(JP203-A)
- U202 pad 5: Net-(JP201-B) -> Net-(JP203-A)
- U202 pad 6: Net-(U202-EN) -> Net-(U202-L2_6)
- U202 pad 7: Net-(U202-EN) -> Net-(U202-L2_6)
- U202 pad 8: Net-(U202-EN) -> Net-(U202-L1_8)
- U202 pad 9: GND -> Net-(U202-L1_8)
- U203 pad 6: Net-(BT201-+) -> Net-(J202-Pin_1)
- U203 pad 8: Net-(BT201-+) -> Net-(J202-Pin_1)
- U301 pad 44: USB.D- -> STM.D-
- U301 pad 45: USB.D+ -> STM.D+
- U401 pad 13: BT.RX -> Net-(U401-UART_RX)
- U401 pad 14: BT.TX -> Net-(U401-UART_TX)
Routing:
- net +3V3: track 0.00 -> 510.4 mm, vias 0 -> 22
- net +5V: track 0.00 -> 131.9 mm, vias 0 -> 3
- net Net-(R508-Pad2): track 0.00 -> 107.0 mm
- net BAT.~{CE}: track 0.00 -> 95.1 mm, vias 0 -> 4
- net SYS.PWR: track 0.00 -> 91.9 mm
- net SD.MISO: track 0.00 -> 90.4 mm, vias 0 -> 3
- net I2C.SCL: track 0.00 -> 89.3 mm, vias 0 -> 3
- net SD.SCLK: track 0.00 -> 88.8 mm, vias 0 -> 3
- net SD.MOSI: track 0.00 -> 88.7 mm, vias 0 -> 3
- net SD.~{CS}: track 0.00 -> 86.8 mm, vias 0 -> 3
- net Net-(R507-Pad2): track 0.00 -> 82.9 mm
- net I2C.SDA: track 0.00 -> 82.2 mm, vias 0 -> 3
- net BAT.GPOUT: track 0.00 -> 81.3 mm, vias 0 -> 3
- net BT.TX: track 0.00 -> 76.7 mm, vias 0 -> 1
- net BAT.EN2: track 0.00 -> 74.0 mm, vias 0 -> 3
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- added copper zone on F.Cu, net /Power Supply Unit/3V_JP
- added copper zone on B.Cu, net GND
- added copper zone on F.Cu, net GND
- added copper zone on F.Cu, net Net-(U204-L1)
- added copper zone on F.Cu, net Net-(U204-L2)
Other:
- board outline added: 130 x 70 mm
