File: PCB/keys.kicad_sch (KiCad schematic)
At the start: 0 parts

Commit message: PCB Update - Minh
Parts:
- added D16, D17, D18, D19, D20, D21, D22, D23, D24, D25, D26, D27, D28, D29, D30, D31: D, symbol Device:D
- added R38, R39, R40, R41, R42, R43, R44, R45, R47: 10k, symbol Device:R
- added SW10, SW11, SW12, SW13, SW14, SW15, SW16, SW17, SW18, SW19, SW20, SW21, SW22, SW6, SW7, SW8, SW9: SW_Push, symbol Switch:SW_Push
Connections:
- new net: D18.2 (A), SW8.1
- new net: R38.2, SW6.2, SW7.2, SW8.2, SW9.2
- new net: D31.2 (A), SW21.1
- new net: R41.2, SW18.2, SW19.2, SW20.2, SW21.2
- new net: D19.1 (K), D23.1 (K), D27.1 (K), D31.1 (K), R45.2
- new net: D19.2 (A), SW9.1
- new net: D23.2 (A), SW13.1
- new net: R39.2, SW10.2, SW11.2, SW12.2, SW13.2
- new net: D18.1 (K), D22.1 (K), D26.1 (K), D30.1 (K), R44.2
- new net: D22.2 (A), SW12.1
- new net: D17.1 (K), D21.1 (K), D25.1 (K), D29.1 (K), R43.2
- new net: D29.2 (A), SW19.1
- new net: D26.2 (A), SW16.1
- new net: R40.2, SW14.2, SW15.2, SW16.2, SW17.2
- new net: D16.1 (K), D20.1 (K), D24.1 (K), D28.1 (K), R42.2
- new net: D25.2 (A), SW15.1
- new net: D30.2 (A), SW20.1
- new net: D20.2 (A), SW10.1
- new net: D21.2 (A), SW11.1
- new net: D24.2 (A), SW14.1
- new net: D17.2 (A), SW7.1
- new net: D16.2 (A), SW6.1
- new net: D27.2 (A), SW17.1
- new net: D28.2 (A), SW18.1
- new net +3V3: R47.2
- new net GND: SW22.2
- new net KEY.COL1: R38.1
- new net KEY.COL2: R39.1
- new net KEY.COL3: R40.1
- new net KEY.COL4: R41.1
- new net KEY.PB0: R47.1, SW22.1
- new net KEY.ROW1: R42.1
- new net KEY.ROW2: R43.1
- new net KEY.ROW3: R44.1
- new net KEY.ROW4: R45.1
Other:
- note added: "Buttons"
- note added: "Schematic Labels"

Commit message: update
Parts:
- removed D16, D17, D18, D19, D20, D21, D22, D23, D24, D25, D26, D27, D28, D29, D30, D31: D, symbol Device:D
- added D501, D502, D503, D504, D505, D506, D507, D508, D509, D510, D511, D512, D513, D514, D515, D516: PMEG4010BEA,115, Diode_SMD:D_SOD-323, symbol Device:D_Schottky
- added R510: 10k, Resistor_SMD:R_0603_1608Metric_Pad0.98x0.95mm_HandSolder, symbol Device:R
- added SW518: SW_Push, Connector_JST:JST_XH_B2B-XH-A_1x02_P2.50mm_Vertical, symbol Switch:SW_Push
- R501: renamed from R42; footprint (none) -> Resistor_SMD:R_0603_1608Metric_Pad0.98x0.95mm_HandSolder; DigiKey Part (none) -> 311-10KGRCT-ND
- R502: renamed from R43; footprint (none) -> Resistor_SMD:R_0603_1608Metric_Pad0.98x0.95mm_HandSolder; DigiKey Part (none) -> 311-10KGRCT-ND
- R503: renamed from R44; footprint (none) -> Resistor_SMD:R_0603_1608Metric_Pad0.98x0.95mm_HandSolder; DigiKey Part (none) -> 311-10KGRCT-ND
- R504: renamed from R45; footprint (none) -> Resistor_SMD:R_0603_1608Metric_Pad0.98x0.95mm_HandSolder; DigiKey Part (none) -> 311-10KGRCT-ND
- R505: renamed from R38; footprint (none) -> Resistor_SMD:R_0603_1608Metric_Pad0.98x0.95mm_HandSolder; DigiKey Part (none) -> 311-10KGRCT-ND
- R506: renamed from R39; footprint (none) -> Resistor_SMD:R_0603_1608Metric_Pad0.98x0.95mm_HandSolder; DigiKey Part (none) -> 311-10KGRCT-ND
- R507: renamed from R40; footprint (none) -> Resistor_SMD:R_0603_1608Metric_Pad0.98x0.95mm_HandSolder; DigiKey Part (none) -> 311-10KGRCT-ND
- R508: renamed from R41; footprint (none) -> Resistor_SMD:R_0603_1608Metric_Pad0.98x0.95mm_HandSolder; DigiKey Part (none) -> 311-10KGRCT-ND
- R509: renamed from R47; footprint (none) -> Resistor_SMD:R_0603_1608Metric_Pad0.98x0.95mm_HandSolder; DigiKey Part (none) -> 311-10KGRCT-ND
- SW501: renamed from SW6; footprint (none) -> Connector_JST:JST_XH_B2B-XH-A_1x02_P2.50mm_Vertical; DigiKey Part (none) -> 455-B2B-XH-A-ND
- SW502: renamed from SW7; footprint (none) -> Connector_JST:JST_XH_B2B-XH-A_1x02_P2.50mm_Vertical; DigiKey Part (none) -> 455-B2B-XH-A-ND
- SW503: renamed from SW8; footprint (none) -> Connector_JST:JST_XH_B2B-XH-A_1x02_P2.50mm_Vertical; DigiKey Part (none) -> 455-B2B-XH-A-ND
- SW504: renamed from SW9; footprint (none) -> Connector_JST:JST_XH_B2B-XH-A_1x02_P2.50mm_Vertical; DigiKey Part (none) -> 455-B2B-XH-A-ND
- SW505: renamed from SW10; footprint (none) -> Connector_JST:JST_XH_B2B-XH-A_1x02_P2.50mm_Vertical; DigiKey Part (none) -> 455-B2B-XH-A-ND
- SW506: renamed from SW11; footprint (none) -> Connector_JST:JST_XH_B2B-XH-A_1x02_P2.50mm_Vertical; DigiKey Part (none) -> 455-B2B-XH-A-ND
- SW507: renamed from SW12; footprint (none) -> Connector_JST:JST_XH_B2B-XH-A_1x02_P2.50mm_Vertical; DigiKey Part (none) -> 455-B2B-XH-A-ND
- SW508: renamed from SW13; footprint (none) -> Connector_JST:JST_XH_B2B-XH-A_1x02_P2.50mm_Vertical; DigiKey Part (none) -> 455-B2B-XH-A-ND
- SW509: renamed from SW14; footprint (none) -> Connector_JST:JST_XH_B2B-XH-A_1x02_P2.50mm_Vertical; DigiKey Part (none) -> 455-B2B-XH-A-ND
- SW510: renamed from SW15; footprint (none) -> Connector_JST:JST_XH_B2B-XH-A_1x02_P2.50mm_Vertical; DigiKey Part (none) -> 455-B2B-XH-A-ND
- SW511: renamed from SW16; footprint (none) -> Connector_JST:JST_XH_B2B-XH-A_1x02_P2.50mm_Vertical; DigiKey Part (none) -> 455-B2B-XH-A-ND
- SW512: renamed from SW17; footprint (none) -> Connector_JST:JST_XH_B2B-XH-A_1x02_P2.50mm_Vertical; DigiKey Part (none) -> 455-B2B-XH-A-ND
- SW513: renamed from SW18; footprint (none) -> Connector_JST:JST_XH_B2B-XH-A_1x02_P2.50mm_Vertical; DigiKey Part (none) -> 455-B2B-XH-A-ND
- SW514: renamed from SW19; footprint (none) -> Connector_JST:JST_XH_B2B-XH-A_1x02_P2.50mm_Vertical; DigiKey Part (none) -> 455-B2B-XH-A-ND
- SW515: renamed from SW20; footprint (none) -> Connector_JST:JST_XH_B2B-XH-A_1x02_P2.50mm_Vertical; DigiKey Part (none) -> 455-B2B-XH-A-ND
- SW516: renamed from SW21; footprint (none) -> Connector_JST:JST_XH_B2B-XH-A_1x02_P2.50mm_Vertical; DigiKey Part (none) -> 455-B2B-XH-A-ND
- SW517: renamed from SW22; footprint (none) -> Connector_JST:JST_XH_B2B-XH-A_1x02_P2.50mm_Vertical; DigiKey Part (none) -> 455-B2B-XH-A-ND
Connections:
- net KEY.COL4 is gone; now on net KEY.COL3: R508.1
- net KEY.ROW4 is gone; now on net KEY.ROW3: R504.1
- net +3V3: now also R510.2
- net GND: now also SW518.2
- net KEY.COL1: now also R506.1; no longer R505.1
- net KEY.COL2: now also R507.1; no longer R506.1
- net KEY.COL3: no longer R507.1
- net KEY.ROW1: now also R502.1; no longer R501.1
- net KEY.ROW2: now also R503.1; no longer R502.1
- net KEY.ROW3: no longer R503.1
- net at SW503.1: now also D503.2 (A)
- net at SW516.1: now also D516.2 (A)
- net at R504.2: now also D504.1 (K), D508.1 (K), D512.1 (K), D516.1 (K)
- net at SW504.1: now also D504.2 (A)
- net at SW508.1: now also D508.2 (A)
- net at R503.2: now also D503.1 (K), D507.1 (K), D511.1 (K), D515.1 (K)
- net at SW507.1: now also D507.2 (A)
- net at R502.2: now also D502.1 (K), D506.1 (K), D510.1 (K), D514.1 (K)
- net at SW514.1: now also D514.2 (A)
- net at SW511.1: now also D511.2 (A)
- net at R501.2: now also D501.1 (K), D505.1 (K), D509.1 (K), D513.1 (K)
- net at SW510.1: now also D510.2 (A)
- net at SW515.1: now also D515.2 (A)
- net at SW505.1: now also D505.2 (A)
- net at SW506.1: now also D506.2 (A)
- net at SW509.1: now also D509.2 (A)
- net at SW502.1: now also D502.2 (A)
- net at SW501.1: now also D501.2 (A)
- net at SW512.1: now also D512.2 (A)
- net at SW513.1: now also D513.2 (A)
- net KEY.PB0 renamed KEY.B17
- new net KEY.B18: R510.1, SW518.1
- new net KEY.COL0: R505.1
- new net KEY.ROW0: R501.1
Other:
- moved on the sheet: R509, SW517

Commit message: Update 90% done
Parts:
- D501, D502, D503, D504, D505, D506, D507, D508, D509, D510, D511, D512, D513, D514, D515, D516: value PMEG4010BEA,115 -> 3757-SS12L_R1_00001CT-ND; footprint Diode_SMD:D_SOD-323 -> Diode_SMD:D_SMA; DigiKey Part 1727-5211-1-ND -> 846-RBS2LAM40BCT-ND; Manufacturer (none) -> Panjit International Inc.; Mfg. Part # (none) -> SS12L_R1_00001; Package (none) -> SOD-128; Supplier (none) -> DigiKey; Supplier Part # (none) -> 3757-SS12L_R1_00001CT-ND
- R501, R502, R503, R504, R505, R506, R507, R508, R509, R510: Manufacturer (none) -> YAGEO; Mfg. Part # (none) -> RC0603JR-0710KL; Package (none) -> 0603; Supplier (none) -> DigiKey; Supplier Part # (none) -> 311-10KGRCT-ND
- SW501, SW502, SW503, SW504, SW505, SW506, SW507, SW508, SW509, SW510, SW511, SW512, SW513, SW514, SW515, SW516, SW517, SW518: Manufacturer (none) -> JST Sales America Inc.; Mfg. Part # (none) -> B2B-XH-A; Package (none) -> B2B-XH-A; Supplier (none) -> DigiKey; Supplier Part # (none) -> 455-B2B-XH-A-ND

Commit message: design 02/17
Parts:
- added R511, R512: 10k, Resistor_SMD:R_0603_1608Metric_Pad0.98x0.95mm_HandSolder, symbol Device:R
Connections:
- net +3V3: now also SW517.1, SW518.1; no longer R509.2, R510.2
- net GND: now also R509.1, R510.1; no longer SW517.2, SW518.2
- net KEY.B17: now also R511.2; no longer R509.1, SW517.1
- net KEY.B18: now also R512.2; no longer R510.1, SW518.1
- new net: R510.2, R512.1, SW518.2
- new net: R509.2, R511.1, SW517.2
Other:
- moved on the sheet: R509, R510, SW517, SW518

Commit message: Update Rev 2
Other:
- company: (none) -> ECE477 - Team 4: KayO
- title: (none) -> Buttons
Changed lines of the file:
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@@
 (kicad_sch (version 20230121) (generator eeschema)
-  (paper "A4")
+  (paper "A3")
+  (title_block
+    (title "Buttons")
+    (date "2024-02-21")
+    (rev "2")
+    (company "ECE477 - Team 4: KayO")
+  )
   (junction (at 88.9 106.68) (diameter 0) (color 0 0 0 0)
   )
@@
     (stroke (width 0) (type default))
   )
-  (bus (pts (xy 228.6 143.51) (xy 232.41 143.51))
+  (bus (pts (xy 352.425 230.505) (xy 356.235 230.505))
     (stroke (width 0) (type default))
   )
@@
     (stroke (width 0) (type default))
   )
-  (rectangle (start 184.15 135.89) (end 281.94 162.56)
+  (rectangle (start 307.975 222.885) (end 405.765 249.555)
     (stroke (width 0) (type default))
     (fill (type none))
@@
     (effects (font (face "KiCad Font") (size 1.27 1.27) (thickness 0.254) bold) (justify left bottom))
   )
-  (text "Schematic Labels" (at 185.42 134.62 0)
+  (text "Schematic Labels" (at 309.245 221.615 0)
     (effects (font (face "KiCad Font") (size 1.27 1.27) (thickness 0.254) bold) (justify left bottom))
   )
@@
     )
   )
-  (global_label "KEY{COL[0..3], ROW[0..3], B17, B18}" (shape bidirectional) (at 228.6 143.51 180) (fields_autoplaced)
-    (effects (font (size 1.27 1.27)) (justify right))
-    (property "Intersheetrefs" "${INTERSHEET_REFS}" (at 188.8828 143.51 0)
+  (global_label "KEY{COL[0..3], ROW[0..3], B17, B18}" (shape bidirectional) (at 352.425 230.505 180) (fields_autoplaced)
+    (effects (font (size 1.27 1.27)) (justify right))
+    (property "Intersheetrefs" "${INTERSHEET_REFS}" (at 312.7078 230.505 0)
       (effects (font (size 1.27 1.27)) (justify right) hide)
     )
@@
     )
   )
-  (hierarchical_label "KEY{COL[0..3], ROW[0..3], B17, B18}" (shape bidirectional) (at 232.41 143.51 0) (fields_autoplaced)
+  (hierarchical_label "KEY{COL[0..3], ROW[0..3], B17, B18}" (shape bidirectional) (at 356.235 230.505 0) (fields_autoplaced)
     (effects (font (size 1.27 1.27)) (justify left))
   )

Commit message: Redesign bluetooth of v2
Parts:
- D501, D502, D503, D504, D505, D506, D507, D508, D509, D510, D511, D512, D513, D514, D515, D516: Package SOD-128 -> (none)
- R501, R502, R503, R504, R505, R506, R507, R508, R509, R510, R511, R512: Package 0603 -> (none)
- SW501, SW502, SW503, SW504, SW505, SW506, SW507, SW508, SW509, SW510, SW511, SW512, SW513, SW514, SW515, SW516, SW517, SW518: Package B2B-XH-A -> (none)
Changed lines of the file:
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@@
-      (effects (font (size 1.27 1.27)) hide)
-    )
-    (property "Package" "B2B-XH-A" (at 106.68 90.17 0)
       (effects (font (size 1.27 1.27)) hide)
     )
@@
       (effects (font (size 1.27 1.27)) hide)
     )
-    (property "Package" "0603" (at 114.3 48.26 0)
-      (effects (font (size 1.27 1.27)) hide)
-    )
     (pin "1")
     (pin "2")
@@
     )
     (property "Supplier Part #" "455-B2B-XH-A-ND" (at 209.55 104.14 0)
-      (effects (font (size 1.27 1.27)) hide)
-    )
-    (property "Package" "B2B-XH-A" (at 209.55 104.14 0)
       (effects (font (size 1.27 1.27)) hide)
     )
@@
       (effects (font (size 1.27 1.27)) hide)
     )
-    (property "Package" "B2B-XH-A" (at 245.11 82.55 0)
-      (effects (font (size 1.27 1.27)) hide)
-    )
     (pin "2")
     (pin "1")
@@
     )
     (property "Supplier Part #" "455-B2B-XH-A-ND" (at 106.68 104.14 0)
-      (effects (font (size 1.27 1.27)) hide)
-    )
-    (property "Package" "B2B-XH-A" (at 106.68 104.14 0)
       (effects (font (size 1.27 1.27)) hide)
     )
@@
       (effects (font (size 1.27 1.27)) hide)
     )
-    (property "Package" "B2B-XH-A" (at 264.16 40.64 0)
-      (effects (font (size 1.27 1.27)) hide)
-    )
     (pin "2")
     (pin "1")
@@
     )
     (property "Supplier Part #" "311-10KGRCT-ND" (at 257.81 46.99 0)
-      (effects (font (size 1.27 1.27)) hide)
-    )
-    (property "Package" "0603" (at 257.81 46.99 0)
       (effects (font (size 1.27 1.27)) hide)
     )
@@
       (effects (font (size 1.27 1.27)) hide)
     )
-    (property "Package" "SOD-128" (at 93.98 104.14 0)
-      (effects (font (size 1.27 1.27)) hide)
-    )
     (pin "1")
     (pin "2")
@@
     )
     (property "Supplier Part #" "455-B2B-XH-A-ND" (at 140.97 104.14 0)
-      (effects (font (size 1.27 1.27)) hide)
-    )
-    (property "Package" "B2B-XH-A" (at 140.97 104.14 0)
       (effects (font (size 1.27 1.27)) hide)
     )
@@
       (effects (font (size 1.27 1.27)) hide)
     )
-    (property "Package" "SOD-128" (at 196.85 76.2 0)
-      (effects (font (size 1.27 1.27)) hide)
-    )
     (pin "1")
     (pin "2")
@@
     )
     (property "Supplier Part #" "455-B2B-XH-A-ND" (at 175.26 90.17 0)
-      (effects (font (size 1.27 1.27)) hide)
-    )
-    (property "Package" "B2B-XH-A" (at 175.26 90.17 0)
       (effects (font (size 1.27 1.27)) hide)
     )
@@
       (effects (font (size 1.27 1.27)) hide)
     )
-    (property "Package" "SOD-128" (at 93.98 76.2 0)
-      (effects (font (size 1.27 1.27)) hide)
-    )
     (pin "1")
     (pin "2")
@@
       (effects (font (size 1.27 1.27)) hide)
     )
-    (property "Package" "0603" (at 76.2 106.68 0)
-      (effects (font (size 1.27 1.27)) hide)
-    )
     (pin "1")
     (pin "2")
@@
     )
     (property "Supplier Part #" "311-10KGRCT-ND" (at 76.2 64.77 0)
-      (effects (font (size 1.27 1.27)) hide)
-    )
-    (property "Package" "0603" (at 76.2 64.77 0)
       (effects (font (size 1.27 1.27)) hide)
     )
@@
       (effects (font (size 1.27 1.27)) hide)
     )
-    (property "Package" "SOD-128" (at 162.56 90.17 0)
-      (effects (font (size 1.27 1.27)) hide)
-    )
     (pin "1")
     (pin "2")
@@
       (effects (font (size 1.27 1.27)) hide)
     )
-    (property "Package" "B2B-XH-A" (at 140.97 90.17 0)
-      (effects (font (size 1.27 1.27)) hide)
-    )
     (pin "2")
     (pin "1")
@@
       (effects (font (size 1.27 1.27)) hide)
     )
-    (property "Package" "B2B-XH-A" (at 209.55 90.17 0)
-      (effects (font (size 1.27 1.27)) hide)
-    )
     (pin "2")
     (pin "1")
@@
     )
     (property "Supplier Part #" "311-10KGRCT-ND" (at 76.2 78.74 0)
-      (effects (font (size 1.27 1.27)) hide)
-    )
-    (property "Package" "0603" (at 76.2 78.74 0)
       (effects (font (size 1.27 1.27)) hide)
     )
@@
       (effects (font (size 1.27 1.27)) hide)
     )
-    (property "Package" "0603" (at 264.16 52.07 0)
-      (effects (font (size 1.27 1.27)) hide)
-    )
     (pin "2")
     (pin "1")
@@
     )
     (property "Supplier Part #" "311-10KGRCT-ND" (at 76.2 92.71 0)
-      (effects (font (size 1.27 1.27)) hide)
-    )
-    (property "Package" "0603" (at 76.2 92.71 0)
       (effects (font (size 1.27 1.27)) hide)
     )
@@
       (effects (font (size 1.27 1.27)) hide)
     )
-    (property "Package" "SOD-128" (at 162.56 104.14 0)
-      (effects (font (size 1.27 1.27)) hide)
-    )
     (pin "1")
     (pin "2")
@@
       (effects (font (size 1.27 1.27)) hide)
     )
-    (property "Package" "SOD-128" (at 93.98 90.17 0)
-      (effects (font (size 1.27 1.27)) hide)
-    )
     (pin "1")
     (pin "2")
@@
       (effects (font (size 1.27 1.27)) hide)
     )
-    (property "Package" "SOD-128" (at 196.85 90.17 0)
-      (effects (font (size 1.27 1.27)) hide)
-    )
     (pin "1")
     (pin "2")
@@
     )
     (property "Supplier Part #" "455-B2B-XH-A-ND" (at 106.68 76.2 0)
-      (effects (font (size 1.27 1.27)) hide)
-    )
-    (property "Package" "B2B-XH-A" (at 106.68 76.2 0)
       (effects (font (size 1.27 1.27)) hide)
     )
@@
       (effects (font (size 1.27 1.27)) hide)
     )
-    (property "Package" "SOD-128" (at 162.56 76.2 0)
-      (effects (font (size 1.27 1.27)) hide)
-    )
     (pin "1")
     (pin "2")
@@
       (effects (font (size 1.27 1.27)) hide)
     )
-    (property "Package" "SOD-128" (at 196.85 104.14 0)
-      (effects (font (size 1.27 1.27)) hide)
-    )
     (pin "1")
     (pin "2")
@@
     )
     (property "Supplier Part #" "455-B2B-XH-A-ND" (at 175.26 104.14 0)
-      (effects (font (size 1.27 1.27)) hide)
-    )
-    (property "Package" "B2B-XH-A" (at 175.26 104.14 0)
       (effects (font (size 1.27 1.27)) hide)
     )
@@
       (effects (font (size 1.27 1.27)) hide)
     )
-    (property "Package" "0603" (at 182.88 48.26 0)
-      (effects (font (size 1.27 1.27)) hide)
-    )
     (pin "1")
     (pin "2")
@@
     )
     (property "Supplier Part #" "455-B2B-XH-A-ND" (at 209.55 76.2 0)
-      (effects (font (size 1.27 1.27)) hide)
-    )
-    (property "Package" "B2B-XH-A" (at 209.55 76.2 0)
       (effects (font (size 1.27 1.27)) hide)
     )
@@
     )
     (property "Supplier Part #" "311-10KGRCT-ND" (at 245.11 93.98 0)
-      (effects (font (size 1.27 1.27)) hide)
-    )
-    (property "Package" "0603" (at 245.11 93.98 0)
       (effects (font (size 1.27 1.27)) hide)
     )
@@
       (effects (font (size 1.27 1.27)) hide)
     )
-    (property "Package" "SOD-128" (at 128.27 104.14 0)
-      (effects (font (size 1.27 1.27)) hide)
-    )
     (pin "1")
     (pin "2")
@@
       (effects (font (size 1.27 1.27)) hide)
     )
-    (property "Package" "SOD-128" (at 162.56 62.23 0)
-      (effects (font (size 1.27 1.27)) hide)
-    )
     (pin "1")
     (pin "2")
@@
       (effects (font (size 1.27 1.27)) hide)
     )
-    (property "Package" "B2B-XH-A" (at 140.97 76.2 0)
-      (effects (font (size 1.27 1.27)) hide)
-    )
     (pin "2")
     (pin "1")
@@
       (effects (font (size 1.27 1.27)) hide)
     )
-    (property "Package" "0603" (at 240.03 88.9 0)
-      (effects (font (size 1.27 1.27)) hide)
-    )
     (pin "2")
     (pin "1")
@@
       (effects (font (size 1.27 1.27)) hide)
     )
-    (property "Package" "B2B-XH-A" (at 175.26 62.23 0)
-      (effects (font (size 1.27 1.27)) hide)
-    )
     (pin "2")
     (pin "1")
@@
       (effects (font (size 1.27 1.27)) hide)
     )
-    (property "Package" "B2B-XH-A" (at 175.26 76.2 0)
-      (effects (font (size 1.27 1.27)) hide)
-    )
     (pin "2")
     (pin "1")
@@
       (effects (font (size 1.27 1.27)) hide)
     )
-    (property "Package" "B2B-XH-A" (at 106.68 62.23 0)
-      (effects (font (size 1.27 1.27)) hide)
-    )
     (pin "2")
     (pin "1")
@@
     )
     (property "Supplier Part #" "455-B2B-XH-A-ND" (at 209.55 62.23 0)
-      (effects (font (size 1.27 1.27)) hide)
-    )
-    (property "Package" "B2B-XH-A" (at 209.55 62.23 0)
       (effects (font (size 1.27 1.27)) hide)
     )
@@
     )
     (property "Supplier Part #" "311-10KGRCT-ND" (at 148.59 48.26 0)
-      (effects (font (size 1.27 1.27)) hide)
-    )
-    (property "Package" "0603" (at 148.59 48.26 0)
       (effects (font (size 1.27 1.27)) hide)
     )
@@
       (effects (font (size 1.27 1.27)) hide)
     )
-    (property "Package" "SOD-128" (at 128.27 90.17 0)
-      (effects (font (size 1.27 1.27)) hide)
-    )
     (pin "1")
     (pin "2")
@@
       (effects (font (size 1.27 1.27)) hide)
     )
-    (property "Package" "SOD-128" (at 196.85 62.23 0)
-      (effects (font (size 1.27 1.27)) hide)
-    )
     (pin "1")
     (pin "2")
@@
       (effects (font (size 1.27 1.27)) hide)
     )
-    (property "Package" "SOD-128" (at 128.27 76.2 0)
-      (effects (font (size 1.27 1.27)) hide)
-    )
     (pin "1")
     (pin "2")
@@
     )
     (property "Supplier Part #" "455-B2B-XH-A-ND" (at 140.97 62.23 0)
-      (effects (font (size 1.27 1.27)) hide)
-    )
-    (property "Package" "B2B-XH-A" (at 140.97 62.23 0)
       (effects (font (size 1.27 1.27)) hide)
     )
@@
       (effects (font (size 1.27 1.27)) hide)
     )
-    (property "Package" "SOD-128" (at 128.27 62.23 0)
-      (effects (font (size 1.27 1.27)) hide)
-    )
     (pin "1")
     (pin "2")
@@
       (effects (font (size 1.27 1.27)) hide)
     )
-    (property "Package" "SOD-128" (at 93.98 62.23 0)
-      (effects (font (size 1.27 1.27)) hide)
-    )
     (pin "1")
     (pin "2")
@@
       (effects (font (size 1.27 1.27)) hide)
     )
-    (property "Package" "0603" (at 217.17 48.26 0)
-      (effects (font (size 1.27 1.27)) hide)
-    )

Commit message: Update PCB Design v2
Parts:
- R501, R502, R503, R504, R505, R506, R507, R508, R509, R510, R511, R512: footprint Resistor_SMD:R_0603_1608Metric_Pad0.98x0.95mm_HandSolder -> Resistor_SMD:R_0805_2012Metric_Pad1.20x1.40mm_HandSolder; Mfg. Part # RC0603JR-0710KL -> RC0805FR-0710KL; Supplier Part # 311-10KGRCT-ND -> 311-10.0KCRCT-ND

Commit message: update
Parts:
- D513: footprint Diode_SMD:D_SMA -> Diode_SMD:D_SOD-123F
Changed lines of the file:
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@@
       (effects (font (size 1.27 1.27)))
     )
-    (property "Footprint" "Diode_SMD:D_SMA" (at 196.85 62.23 0)
+    (property "Footprint" "Diode_SMD:D_SOD-123F" (at 196.85 62.23 0)
       (effects (font (size 1.27 1.27)) hide)
     )
